File: hw/breakout_pcb/hats/backpower_eeprom_rpibout.brd (EAGLE design)
At the start: 65 x 30 mm, 31 parts, among them IC2 DMMT5401, U1 PTR08060W, U2 BSS138BKS, X1 22-23-2021

Commit message: Add files via upload
Parts:
- removed IC2: DMMT5401, GPIO Split Protector with Console:DIODES_INC_BY_ELEMENT14_BATCH_1_DMMT5401
- removed U$1: DMG2305UX, rpibout:SOT23-3
- removed U$2: MMDT5401, rpibout:SOT363
- removed U$4: EEPROM_CAT24C32WI-GT3, rpibout:SOIC-8
- removed X1: 22-23-2021, con-molex:22-23-2021
- added DMG2305: DMG2305UX, rpibout:SOT23-3
- added EEPROM: EEPROM_CAT24C32WI-GT3, rpibout:SOIC-8
- added JP1: (no value), pinhead:1X02
- added JP2: (no value), jumper:JP1
- added MMDT5401: MMDT5401, rpibout:SOT363
- moved C3 106.0 mm to (-27.9, 68.6), flipped to the top, turned to 0 degrees
- moved U2 105.3 mm to (-48.3, 61.0), turned to 0 degrees
- moved C4 96.9 mm to (-33.0, 68.6), flipped to the top
- moved R4 96.1 mm to (-33.0, 73.7), flipped to the top
- moved H1 95.8 mm to (-27.9, 61.0)
- moved R5 95.7 mm to (-38.1, 73.7), flipped to the top
- moved LEDMATRIX 92.8 mm to (-27.9, 3.81), turned to 0 degrees
- moved C2 91.3 mm to (-63.5, 40.6)
- moved C5 87.9 mm to (-38.1, 68.6), flipped to the top, turned to 0 degrees
- moved R1 86.5 mm to (-43.2, 68.6), flipped to the top, turned to 0 degrees
- moved R3 84.1 mm to (-27.9, 73.7), flipped to the top
- moved IMU 84.0 mm to (-41.9, 43.2), turned to 0 degrees
- moved ENC2 79.3 mm to (-30.5, 43.2), turned to 0 degrees
- moved R2 78.7 mm to (-22.9, 73.7), flipped to the top
- moved U1 78.7 mm to (-57.1, 27.9), turned to 0 degrees
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Connections:
- removed net +5V_SUPPLY: C2.+, C3.1, C4.1, U$2.4, U1.P4
- removed net N$8: X1.1
- new net VOUT: C2.+, C3.1, C4.1, DMG2305.3, MMDT5401.4, U1.P4
- net +3V3: now also EEPROM.8; no longer U$4.8
- net +5V: now also DMG2305.2, MMDT5401.1; no longer U$1.2, U$2.1
- net GND: now also EEPROM.1, EEPROM.2, EEPROM.3, EEPROM.4, JP1.1, JP2.1; no longer U$4.1, U$4.2, U$4.3, U$4.4
- net N$1: now also MMDT5401.2, MMDT5401.3, MMDT5401.5; no longer U$2.2, U$2.3, U$2.5
- net N$3: now also DMG2305.1, MMDT5401.6; no longer U$1.1, U$2.6
- net N$5: now also EEPROM.5; no longer U$4.5
- net N$7: now also EEPROM.6; no longer U$4.6
- net N$9: now also EEPROM.7, JP1.2, JP2.2; no longer U$4.7, X1.2
Routing:
- net GPIO12: track 49.0 -> 0.00 mm, vias 2 -> 0
- net GPIO13: track 47.6 -> 0.00 mm, vias 2 -> 0
- net +3V3: track 47.1 -> 0.00 mm
- net GPIO16: track 46.8 -> 0.00 mm, vias 2 -> 0
- net GPIO19: track 45.7 -> 0.00 mm, vias 2 -> 0
- net SCL3V3: track 45.3 -> 0.00 mm, vias 2 -> 0
- net GPIO5: track 42.2 -> 0.00 mm, vias 2 -> 0
- net GPIO6: track 42.1 -> 0.00 mm, vias 2 -> 0
- net SDA3V3: track 40.6 -> 0.00 mm, vias 2 -> 0
- net GND: track 19.9 -> 0.00 mm, vias 1 -> 0
- net SCL5V: track 19.3 -> 0.00 mm, vias 1 -> 0
- net SDA5V: track 17.9 -> 0.00 mm, vias 1 -> 0
- net N$2: track 3.84 -> 0.00 mm
- removed copper zone on layer 16, net +5V
- removed copper zone on layer 1, net GND
- removed copper zone on layer 16, net VBATT
Other:
- board size 65 x 30 mm -> 160 x 100 mm
- board text removed: "1"
- board text removed: "Raspberry Pi Car Breakout Board v1.1 WashU ESE Dept Nov 2016"
