File: hw/breakout_pcb/pcb.sch (EAGLE design)
At the start: 108 parts, among them U1 BTN8982TA, U10 BSS138BKS, U2 BTN8982TA, U3 BTN8982TA, U4 BTN8982TA, U5 BTN8982TA, U6 BTN8982TA, U7 PTR08060W

Commit message: Add files via upload
Parts:
- U1, U2, U3, U4, U5, U6: device BTN8982TA:BTN8982TA -> rpibout:BTN8982TA

Commit message: Add files via upload
Parts:
- added MOTOR_CONN1, MOTOR_CONN2: ULTRAFIT_3CIRC, rpibout:ULTRAFIT_3CIRC
Connections:
- net OUT1: now also MOTOR_CONN1.P1
- net OUT2: now also MOTOR_CONN1.P2
- net OUT3: now also MOTOR_CONN1.P3
- net OUT4: now also MOTOR_CONN2.P1
- net OUT5: now also MOTOR_CONN2.P2
- net OUT6: now also MOTOR_CONN2.P3
Changed lines of the file:
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@@
 <part name="U5" library="rpibout" deviceset="BTN8982TA" device=""/>
 <part name="U6" library="rpibout" deviceset="BTN8982TA" device=""/>
+<part name="MOTOR_CONN1" library="rpibout" deviceset="ULTRAFIT_3CIRC" device=""/>
+<part name="MOTOR_CONN2" library="rpibout" deviceset="ULTRAFIT_3CIRC" device=""/>
 </parts>
 <sheets>
@@
 <instance part="U5" gate="G$1" x="213.36" y="-10.16"/>
 <instance part="U6" gate="G$1" x="213.36" y="-58.42"/>
+<instance part="MOTOR_CONN1" gate="G$1" x="137.16" y="-15.24"/>
+<instance part="MOTOR_CONN2" gate="G$1" x="304.8" y="-12.7"/>
 </instances>
 <busses>
@@
 <pinref part="U1" gate="G$1" pin="OUT2"/>
 </segment>
+<segment>
+<pinref part="MOTOR_CONN1" gate="G$1" pin="P1"/>
+<wire x1="137.16" y1="-15.24" x2="127" y2="-15.24" width="0.1524" layer="91"/>
+<label x="127" y="-15.24" size="1.778" layer="95"/>
+</segment>
 </net>
 <net name="OUT2" class="0">
@@
 <pinref part="U2" gate="G$1" pin="OUT2"/>
 </segment>
+<segment>
+<pinref part="MOTOR_CONN1" gate="G$1" pin="P2"/>
+<wire x1="137.16" y1="-17.78" x2="127" y2="-17.78" width="0.1524" layer="91"/>
+<label x="127" y="-17.78" size="1.778" layer="95"/>
+</segment>
 </net>
 <net name="OUT3" class="0">
@@
 <pinref part="U3" gate="G$1" pin="OUT2"/>
 </segment>
+<segment>
+<pinref part="MOTOR_CONN1" gate="G$1" pin="P3"/>
+<wire x1="137.16" y1="-20.32" x2="127" y2="-20.32" width="0.1524" layer="91"/>
+<label x="127" y="-20.32" size="1.778" layer="95"/>
+</segment>
 </net>
 <net name="N$21" class="0">
@@
 <pinref part="U4" gate="G$1" pin="OUT2"/>
 </segment>
+<segment>
+<pinref part="MOTOR_CONN2" gate="G$1" pin="P1"/>
+<wire x1="304.8" y1="-12.7" x2="297.18" y2="-12.7" width="0.1524" layer="91"/>
+<label x="294.64" y="-12.7" size="1.778" layer="95"/>
+</segment>
 </net>
 <net name="OUT5" class="0">
@@
 <pinref part="U5" gate="G$1" pin="OUT2"/>
 </segment>
+<segment>
+<pinref part="MOTOR_CONN2" gate="G$1" pin="P2"/>
+<wire x1="304.8" y1="-15.24" x2="297.18" y2="-15.24" width="0.1524" layer="91"/>
+<label x="294.64" y="-15.24" size="1.778" layer="95"/>
+</segment>
 </net>
 <net name="OUT6" class="0">
@@
 <pinref part="U6" gate="G$1" pin="OUT2"/>
 </segment>
-</net>
+<segment>
+<pinref part="MOTOR_CONN2" gate="G$1" pin="P3"/>
+<wire x1="304.8" y1="-17.78" x2="297.18" y2="-17.78" width="0.1524" layer="91"/>
+<label x="294.64" y="-17.78" size="1.778" layer="95"/>
+</segment>
+</net>

Commit message: Add files via upload
Connections:
- new net N$2: R26.2, R27.2
- new net N$3: R28.2, R29.2
- net +3V3: no longer R26.2, R27.2, R28.2, R29.2
Changed lines of the file:
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@@
 <part name="GND36" library="supply1" deviceset="GND" device=""/>
 <part name="GND37" library="supply1" deviceset="GND" device=""/>
-<part name="+3V5" library="supply1" deviceset="+3V3" device=""/>
-<part name="+3V6" library="supply1" deviceset="+3V3" device=""/>
 <part name="IMU" library="con-molex" deviceset="22-23-2041" device=""/>
 <part name="GND40" library="supply1" deviceset="GND" device=""/>
@@
 <part name="MOTOR_CONN1" library="rpibout" deviceset="ULTRAFIT_3CIRC" device=""/>
 <part name="MOTOR_CONN2" library="rpibout" deviceset="ULTRAFIT_3CIRC" device=""/>
+<part name="P+12" library="supply1" deviceset="+5V" device=""/>
+<part name="P+13" library="supply1" deviceset="+5V" device=""/>
 </parts>
 <sheets>
@@
 <instance part="GND36" gate="1" x="233.68" y="134.62"/>
 <instance part="GND37" gate="1" x="233.68" y="104.14"/>
-<instance part="+3V5" gate="G$1" x="220.98" y="162.56"/>
-<instance part="+3V6" gate="G$1" x="220.98" y="132.08"/>
 <instance part="IMU" gate="-1" x="299.72" y="114.3" smashed="yes">
 <attribute name="NAME" x="302.26" y="113.538" size="1.524" layer="95"/>
@@
 <instance part="MOTOR_CONN1" gate="G$1" x="137.16" y="-15.24"/>
 <instance part="MOTOR_CONN2" gate="G$1" x="304.8" y="-12.7"/>
+<instance part="P+12" gate="1" x="220.98" y="162.56"/>
+<instance part="P+13" gate="1" x="220.98" y="132.08"/>
 </instances>
 <busses>
@@
 <net name="+3V3" class="0">
 <segment>
-<pinref part="R26" gate="G$1" pin="2"/>
-<pinref part="R27" gate="G$1" pin="2"/>
-<wire x1="218.44" y1="157.48" x2="220.98" y2="157.48" width="0.1524" layer="91"/>
-<pinref part="+3V5" gate="G$1" pin="+3V3"/>
-<wire x1="220.98" y1="157.48" x2="223.52" y2="157.48" width="0.1524" layer="91"/>
-<wire x1="220.98" y1="160.02" x2="220.98" y2="157.48" width="0.1524" layer="91"/>
-<junction x="220.98" y="157.48"/>
-</segment>
-<segment>
-<pinref part="R28" gate="G$1" pin="2"/>
-<pinref part="R29" gate="G$1" pin="2"/>
-<wire x1="218.44" y1="127" x2="220.98" y2="127" width="0.1524" layer="91"/>
-<pinref part="+3V6" gate="G$1" pin="+3V3"/>
-<wire x1="220.98" y1="127" x2="223.52" y2="127" width="0.1524" layer="91"/>
-<wire x1="220.98" y1="129.54" x2="220.98" y2="127" width="0.1524" layer="91"/>
-<junction x="220.98" y="127"/>
-</segment>
-<segment>
 <pinref part="IMU" gate="-4" pin="S"/>
 <wire x1="297.18" y1="106.68" x2="289.56" y2="106.68" width="0.1524" layer="91"/>
@@
 </segment>
 </net>
+<net name="N$2" class="0">
+<segment>
+<pinref part="R26" gate="G$1" pin="2"/>
+<pinref part="R27" gate="G$1" pin="2"/>
+<wire x1="218.44" y1="157.48" x2="220.98" y2="157.48" width="0.1524" layer="91"/>
+<wire x1="220.98" y1="157.48" x2="223.52" y2="157.48" width="0.1524" layer="91"/>
+<wire x1="220.98" y1="160.02" x2="220.98" y2="157.48" width="0.1524" layer="91"/>
+<junction x="220.98" y="157.48"/>
+</segment>
+</net>
+<net name="N$3" class="0">
+<segment>
+<pinref part="R28" gate="G$1" pin="2"/>
+<pinref part="R29" gate="G$1" pin="2"/>
+<wire x1="218.44" y1="127" x2="220.98" y2="127" width="0.1524" layer="91"/>
+<wire x1="220.98" y1="127" x2="223.52" y2="127" width="0.1524" layer="91"/>
+<wire x1="220.98" y1="129.54" x2="220.98" y2="127" width="0.1524" layer="91"/>
+<junction x="220.98" y="127"/>
+</segment>
+</net>

Commit message: minor editorial changes to pcb.sch
Other:
- moved on the sheet: C31, HALL5-1, HALL5-2, HALL5-3, R33, R35, R39, R41

Commit message: Add files via upload
Parts:
- removed J1: (no value), pinhead:PINHD-2X20
- removed U$2: ARDUINO_MEGA, rpibout:ARDUINO_MEGA
- added 0~1, 0~7: 2.54-8P-female, Connector:HEADER-8P-60/35MIL
- added C38: 0.1u, resistor:C-USC1206
- added D38~, D46~: DNP, Connector:HEADER-8P-60/35MIL
- added EEPROM: EEPROM_CAT24C32WI-GT3, rpibout:EEPROM_CAT24C32WI-GT3
- added I2C: 2.54-4P-female, Connector:HEADER-4P-60/35MIL
- added ISP: CK_2X3, Connector:HEADER-2X3P-60/35MIL
- added J11: 2.54-6P-female, Connector:HEADER-6P-60/35MIL
- added J2: (no value), pinhead:PINHD-2X20
- added JUMPER: 02JUMPER, rpibout:02JUMPER
- added R45, R46: 3.9k, resistor:R-US_R1206
- added R47: 1k, resistor:R-US_R1206
Connections:
- removed net D22: ENC1-3.S, R26.1, U$2.22
- removed net D23: ENC1-4.S, R27.1, U$2.23
- removed net D24: ENC2-3.S, R28.1, U$2.24
- removed net D25: ENC2-4.S, R29.1, U$2.25
- removed net D26: R1.1, R5.1, R9.1, U$2.26
- removed net D27: R13.1, R18.1, R22.1, U$2.27
- removed net D28: HALL1-3.S, R39.1, U$2.28
- removed net D29: HALL2-3.S, R40.1, U$2.29
- removed net D30: HALL3-3.S, R41.1, U$2.30
- removed net D31: HALL4-3.S, R33.1, U$2.31
- removed net D32: HALL5-3.S, R34.1, U$2.32
- removed net D33: HALL6-3.S, R35.1, U$2.33
- removed net IOREF: U$2.IOREF
- removed net RESET: U$2.RESET
- new net 3V3: J11.5
- new net D38: D38~.1, ENC1-3.S, R26.1
- new net D39: D38~.2, ENC1-4.S, R27.1
- new net D40: D38~.3, ENC2-3.S, R28.1
- new net D41: D38~.4, ENC2-4.S, R29.1
- new net D42: D38~.5, R1.1, R5.1, R9.1
- new net D43: D38~.6, HALL1-3.S, R39.1
- new net D44: D38~.7, HALL2-3.S, R40.1
- new net D45: D38~.8, HALL3-3.S, R41.1
- new net D46: D46~.1, R13.1, R18.1, R22.1
- new net D47: D46~.2, HALL4-3.S, R33.1
- new net D48: D46~.3, HALL5-3.S, R34.1
- new net D49: D46~.4, HALL6-3.S, R35.1
- new net MEGASCK: D46~.7, ISP.2
- new net N$10: EEPROM.SDA, J2.27, R45.1
- new net N$12: EEPROM.WP, JUMPER.P2, R47.1
- new net N$7: EEPROM.SCL, J2.28, R46.1
- new net PWR_IN: J11.1
- new net RESET_1280: ISP.3, J11.6
- new net VCC: I2C.P$1, ISP.6
- net +3V3: now also C38.1, EEPROM.VCC, J2.17, R45.2, R46.2, R47.2; no longer U$2.3.3V
- net +5V: now also J11.4, J2.2, J2.4; no longer J1.2, J1.4, U$2.5V@0, U$2.5V@1, U$2.5V@2
- net GND: now also C38.2, EEPROM.A0, EEPROM.A1, EEPROM.A2, EEPROM.VSS, I2C.P$2, ISP.4, J11.2, J11.3, J2.14, J2.20, J2.25, J2.30, J2.34, J2.39, J2.6, JUMPER.P1; no longer J1.14, J1.20, J1.25, J1.30, J1.34, J1.39, J1.6, U$2.GND@0, U$2.GND@1, U$2.GND@2, U$2.GND@3, U$2.GND@4
- net MEGAA2: now also 0~1.3; no longer U$2.A2
- net MEGAA3: now also 0~1.4; no longer U$2.A3
- net MEGAA4: now also 0~1.5; no longer U$2.A4
- net MEGAA5: now also 0~1.6; no longer U$2.A5
- net MEGAA6: now also 0~1.7; no longer U$2.A6
- net MEGAA7: now also 0~1.8; no longer U$2.A7
- net MEGAMISO: now also D46~.5, ISP.1; no longer U$2.50
- net MEGAMOSI: now also D46~.6, ISP.5; no longer U$2.51
- net MEGASCL: now also I2C.P$3; no longer U$2.21(SCL)
- net MEGASCLK: no longer U$2.52
- net MEGASDA: now also I2C.P$4; no longer U$2.20(SDA)
- net PWM2: now also 0~7.3; no longer U$2.2
- net PWM3: now also 0~7.4; no longer U$2.3
- net PWM4: now also 0~7.5; no longer U$2.4
- net PWM5: now also 0~7.6; no longer U$2.5
- net PWM6: now also 0~7.7; no longer U$2.6
- net PWM7: now also 0~7.8; no longer U$2.7
- net RPIMISO: now also J2.21; no longer J1.21
- net RPIMOSI: now also J2.19; no longer J1.19
- net RPISCLK: now also J2.23; no longer J1.23
Other:
- note added: "56"
- note added: "57"
- note added: "58"
- note added: "59"
- note added: "60"
- note added: "61"
- note added: "A2"
- note added: "A3"
- note added: "A4"
- note added: "A5"
- note added: "A6"
- note added: "A7"
- note added: "D2"
- note added: "D3"
- note added: "D38"
- note added: "D39"
- note added: "D4"
- note added: "D40"
- note added: "D41"
- note added: "D42"
- note added: "D43"
- note added: "D44"
- note added: "D45"
- note added: "D46"
- note added: "D47"
- note added: "D48"
- note added: "D49"
- note added: "D5"
- note added: "D50"
- note added: "D51"
- note added: "D52"
- note added: "D6"
- note added: "D7"
- moved on the sheet: BATT1, C16, C17, C31, C34, C35, C36, C37, D1, D2, DMG2305, HALL5-1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

Commit message: Add files via upload
Parts:
- removed ISP: CK_2X3, Connector:HEADER-2X3P-60/35MIL
Connections:
- net GND: no longer ISP.4
- net MEGAMISO: no longer ISP.1
- net MEGAMOSI: no longer ISP.5
- net MEGASCK: no longer ISP.2
- net RESET_1280: no longer ISP.3
- net VCC: no longer ISP.6
Changed lines of the file:
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@@
 <part name="P+13" library="supply1" deviceset="+5V" device=""/>
 <part name="0~7" library="Connector" deviceset="HEADER-8P" device="-60/35MIL" value="2.54-8P-female"/>
-<part name="ISP" library="Connector" deviceset="HEADER-2X3P" device="-60/35MIL" value="CK_2X3"/>
 <part name="J11" library="Connector" deviceset="HEADER-6P" device="-60/35MIL" value="2.54-6P-female"/>
 <part name="D38~" library="Connector" deviceset="HEADER-8P" device="-60/35MIL" value="DNP"/>
@@
 <instance part="P+13" gate="1" x="220.98" y="132.08"/>
 <instance part="0~7" gate="J" x="154.94" y="125.73" rot="R180"/>
-<instance part="ISP" gate="J" x="140.97" y="147.32"/>
 <instance part="J11" gate="J" x="102.87" y="130.81" rot="R180"/>
 <instance part="D38~" gate="J" x="154.94" y="100.33" rot="MR0"/>
@@
 </segment>
 <segment>
-<wire x1="165.1" y1="144.78" x2="148.59" y2="144.78" width="0.1524" layer="91"/>
-<label x="149.86" y="144.78" size="1.778" layer="95"/>
-<pinref part="ISP" gate="J" pin="4"/>
-</segment>
-<segment>
 <wire x1="107.95" y1="76.2" x2="132.08" y2="76.2" width="0.1524" layer="91"/>
 <label x="113.03" y="76.2" size="1.778" layer="95"/>
@@
 <pinref part="D46~" gate="J" pin="6"/>
 </segment>
-<segment>
-<wire x1="165.1" y1="147.32" x2="148.59" y2="147.32" width="0.1524" layer="91"/>
-<label x="149.86" y="147.32" size="1.778" layer="95"/>
-<pinref part="ISP" gate="J" pin="5"/>
-</segment>
 </net>
 <net name="MEGAMISO" class="0">
@@
 <label x="162.56" y="74.93" size="1.778" layer="95"/>
 <pinref part="D46~" gate="J" pin="5"/>
-</segment>
-<segment>
-<wire x1="118.11" y1="149.86" x2="133.35" y2="149.86" width="0.1524" layer="91"/>
-<label x="119.38" y="149.86" size="1.778" layer="95"/>
-<pinref part="ISP" gate="J" pin="1"/>
 </segment>
 </net>
@@
 <pinref part="J11" gate="J" pin="6"/>
 </segment>
-<segment>
-<wire x1="118.11" y1="144.78" x2="133.35" y2="144.78" width="0.1524" layer="91"/>
-<label x="119.38" y="144.78" size="1.778" layer="95"/>
-<pinref part="ISP" gate="J" pin="3"/>
-</segment>
 </net>
 <net name="VCC" class="0">
@@
 <label x="113.03" y="73.66" size="1.778" layer="95"/>
 <pinref part="I2C" gate="G$1" pin="P$1"/>
-</segment>
-<segment>
-<wire x1="165.1" y1="149.86" x2="148.59" y2="149.86" width="0.1524" layer="91"/>
-<label x="149.86" y="149.86" size="1.778" layer="95"/>
-<pinref part="ISP" gate="J" pin="6"/>
 </segment>
 </net>
@@
 <pinref part="D46~" gate="J" pin="7"/>
 </segment>
-<segment>
-<wire x1="118.11" y1="147.32" x2="133.35" y2="147.32" width="0.1524" layer="91"/>
-<label x="119.38" y="147.32" size="1.778" layer="95"/>
-<pinref part="ISP" gate="J" pin="2"/>
-</segment>
-</net>
+</net>
