File: hw/motorcontrol/motorcontrol.sch (EAGLE design)
At the start: 82 parts, among them U1 BTN8982TA, U10 BSS138BKS, U2 BTN8982TA, U3 BTN8982TA, U7 PTR08060W

Commit message: .\motorcontrol.sch
Parts:
- removed R32, R42: 10k, resistor:R-US_R1206
- added C22: 0.1u, resistor:C-USC1206
- added C23, C24: 100n, resistor:C-USC1206
- added R13: 1M, resistor:R-US_R1206
- added U$4: SWITCH, rpibout:SWITCH
- U$5: value BSS138BKS -> ADG3304; device rpibout:BSS138BKS -> rpibout:ADG3304
Connections:
- removed net ATMEGASCLK: R44.1, U$5T1.D
- removed net N$14: R48.1, U$2./RESET
- removed net N$2: R26.2, R27.2
- new net IMUSCL: IMU-1.S, R44.1, U10T1.D
- new net IMUSDA: IMU-2.S, R31.1, U10T2.D
- new net N$16: C18.1, R13.1, U$2.XTAL2, U$3.1
- new net RPISCK: U$5.A3
- net +3V3: now also C23.1, R31.2, R44.2, U$5.VCCA; no longer R30.2, R32.2, R43.2, U$5T1.G, U10T1.G, U10T2.G
- net +5V: now also C22.1, C24.1, R26.2, R27.2, R30.2, R43.2, U$5.EN, U$5.VCCY, U10T1.G, U10T2.G; no longer R31.2, R42.2, R44.2
- net ATMEGAMISO: now also U$5.Y2; no longer R31.1, U10T2.D
- net ATMEGAMOSI: now also U$5.Y1; no longer R42.1, U10T1.D
- net ATMEGASCK: now also U$5.Y3
- net ATMEGASCL: now also R43.1, U10T1.S; no longer IMU-1.S
- net ATMEGASDA: now also R30.1, U10T2.S; no longer IMU-2.S
- net GND: now also C23.2, C24.2, U$4.1, U$5.GND
- net N$3: now also R13.2
- net N$8: now also C22.2, J2.12, R48.1, U$2./RESET, U$4.2; no longer C18.1, U$2.XTAL2, U$3.1
- net RPIMISO: now also U$5.A2; no longer R30.1, U10T2.S
- net RPIMOSI: now also U$5.A1; no longer R32.1, U10T1.S
- net RPISCLK: no longer R43.1, U$5T1.S
Other:
- note removed: "Logic Level Converter"
- moved on the sheet: C18, C19, C20, C21, C33, C38, EEPROM, ENC1-1, ENC1-2, ENC1-3, ENC1-4, IMU-1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

Commit message: .\motorcontrol.sch
Parts:
- added U$6: SWITCH, rpibout:SWITCH
Connections:
- new net N$14: U$2.AVCC, U$2.AVCC1, U$2.VCC, U$2.VCC1, U$6.1
- net +5V: now also U$6.2; no longer U$2.AVCC, U$2.AVCC1, U$2.VCC, U$2.VCC1
Changed lines of the file:
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@@
 <part name="GND41" library="supply1" deviceset="GND" device=""/>
 <part name="GND42" library="supply1" deviceset="GND" device=""/>
-<part name="P+10" library="supply1" deviceset="+5V" device=""/>
 <part name="R48" library="resistor" deviceset="R-US_" device="R1206" value="10k"/>
 <part name="SERVO_MOTOR" library="rpibout" deviceset="ULTRAFIT_3CIRC" device=""/>
@@
 <part name="GND25" library="supply1" deviceset="GND" device=""/>
 <part name="GND26" library="supply1" deviceset="GND" device=""/>
+<part name="U$6" library="rpibout" deviceset="SWITCH" device=""/>
+<part name="P+6" library="supply1" deviceset="+5V" device=""/>
 </parts>
 <sheets>
@@
 <instance part="GND41" gate="1" x="27.94" y="63.5"/>
 <instance part="GND42" gate="1" x="88.9" y="124.46"/>
-<instance part="P+10" gate="1" x="25.4" y="149.86"/>
 <instance part="R48" gate="G$1" x="7.62" y="149.86" smashed="yes" rot="R90">
 <attribute name="NAME" x="6.1214" y="148.59" size="1.778" layer="95" rot="R90"/>
@@
 <instance part="GND25" gate="1" x="127" y="63.5"/>
 <instance part="GND26" gate="1" x="149.86" y="96.52"/>
+<instance part="U$6" gate="G$1" x="25.4" y="154.94" rot="R90"/>
+<instance part="P+6" gate="1" x="25.4" y="165.1"/>
 </instances>
 <busses>
@@
 </segment>
 <segment>
-<pinref part="U$2" gate="G$1" pin="VCC"/>
-<pinref part="P+10" gate="1" pin="+5V"/>
-<wire x1="30.48" y1="132.08" x2="25.4" y2="132.08" width="0.1524" layer="91"/>
-<wire x1="25.4" y1="132.08" x2="25.4" y2="147.32" width="0.1524" layer="91"/>
-<pinref part="U$2" gate="G$1" pin="VCC1"/>
-<wire x1="30.48" y1="129.54" x2="25.4" y2="129.54" width="0.1524" layer="91"/>
-<wire x1="25.4" y1="129.54" x2="25.4" y2="132.08" width="0.1524" layer="91"/>
-<junction x="25.4" y="132.08"/>
-<pinref part="U$2" gate="G$1" pin="AVCC"/>
-<wire x1="30.48" y1="124.46" x2="25.4" y2="124.46" width="0.1524" layer="91"/>
-<wire x1="25.4" y1="124.46" x2="25.4" y2="129.54" width="0.1524" layer="91"/>
-<junction x="25.4" y="129.54"/>
-<pinref part="U$2" gate="G$1" pin="AVCC1"/>
-<wire x1="30.48" y1="121.92" x2="25.4" y2="121.92" width="0.1524" layer="91"/>
-<wire x1="25.4" y1="121.92" x2="25.4" y2="124.46" width="0.1524" layer="91"/>
-<junction x="25.4" y="124.46"/>
-</segment>
-<segment>
 <pinref part="SERVO_MOTOR" gate="G$1" pin="P1"/>
 <wire x1="223.52" y1="157.48" x2="213.36" y2="157.48" width="0.1524" layer="91"/>
@@
 <wire x1="165.1" y1="101.6" x2="170.18" y2="101.6" width="0.1524" layer="91"/>
 <junction x="170.18" y="101.6"/>
+</segment>
+<segment>
+<pinref part="U$6" gate="G$1" pin="2"/>
+<pinref part="P+6" gate="1" pin="+5V"/>
+<wire x1="25.4" y1="162.56" x2="25.4" y2="160.02" width="0.1524" layer="91"/>
 </segment>
 </net>
@@
 </segment>
 </net>
+<net name="N$14" class="0">
+<segment>
+<pinref part="U$2" gate="G$1" pin="VCC"/>
+<wire x1="30.48" y1="132.08" x2="25.4" y2="132.08" width="0.1524" layer="91"/>
+<wire x1="25.4" y1="132.08" x2="25.4" y2="149.86" width="0.1524" layer="91"/>
+<pinref part="U$2" gate="G$1" pin="VCC1"/>
+<wire x1="30.48" y1="129.54" x2="25.4" y2="129.54" width="0.1524" layer="91"/>
+<wire x1="25.4" y1="129.54" x2="25.4" y2="132.08" width="0.1524" layer="91"/>
+<junction x="25.4" y="132.08"/>
+<pinref part="U$2" gate="G$1" pin="AVCC"/>
+<wire x1="30.48" y1="124.46" x2="25.4" y2="124.46" width="0.1524" layer="91"/>
+<wire x1="25.4" y1="124.46" x2="25.4" y2="129.54" width="0.1524" layer="91"/>
+<junction x="25.4" y="129.54"/>
+<pinref part="U$2" gate="G$1" pin="AVCC1"/>
+<wire x1="30.48" y1="121.92" x2="25.4" y2="121.92" width="0.1524" layer="91"/>
+<wire x1="25.4" y1="121.92" x2="25.4" y2="124.46" width="0.1524" layer="91"/>
+<junction x="25.4" y="124.46"/>
+<pinref part="U$6" gate="G$1" pin="1"/>
+</segment>
+</net>
