File: hw/motorcontrol/motorcontrol.sch (EAGLE design)
At the start: 87 parts, among them U1 BTN8982TA, U10 BSS138BKS, U11 DMG2305UX, U2 BTN8982TA, U3 BTN8982TA, U4 CAT24C32WI-GT3, U5 ADG3304, U6 MMDT5401, U7 PTR08060W, U8 IPD90P03P4L_04, U9 ATMEGA32U4

Commit message: motorcontrol schematic should be ready
Parts:
- removed ENC1: 22-23-2041, con-molex:22-23-2041
- removed MOTOR_CONN1, SERVO_MOTOR: ULTRAFIT_3CIRC, rpibout:ULTRAFIT_3CIRC
- removed U$3: CRYSTAL, rpibout:CRYSTAL
- removed U$4: SWITCH, rpibout:SWITCH
- added C25, C26, C27, C28, C29: 1u, resistor:C-USC1206
- added ENCODER: 22-23-2041, con-molex:22-23-2041
- added J3: SWITCH, rpibout:SWITCH
- added J4: ULTRAFIT_3CIRC, rpibout:ULTRAFIT_3CIRC
- added SERVO: 22-23-2031, con-molex:22-23-2031
- added U12: CRYSTAL, rpibout:CRYSTAL
- C23, C24: value 100n -> 0.1u
- R26, R27: value (none) -> 3.9k
- R30, R31, R43, R44: value 10k -> 3.9k
- U8: value IPD90P03P4L_04 -> IPD90P03P4L-04; device rpibout:IPD90P03P4L_04 -> rpibout:IPD90P03P4L-04
Connections:
- net RPISCL renamed RPIROMSCL
- net RPISDA renamed RPIROMSDA
- new net ATMEGARESET: C22.2, J3.2, R48.1, U5.Y4, U9./RESET
- net +3V3: now also J2.1
- net +5V: now also C25.1, C26.1, C27.1, C28.1, C29.1, ENCODER-1.S, SERVO-1.S, U6T2.E; no longer ENC1-1.S, SERVO_MOTOR.P1, U6G$2.E
- net D13: now also SERVO-2.S; no longer SERVO_MOTOR.P2
- net D4: now also ENCODER-3.S; no longer ENC1-3.S
- net D5: now also ENCODER-4.S; no longer ENC1-4.S
- net GND: now also C25.2, C26.2, C27.2, C28.2, C29.2, ENCODER-2.S, J2.9, J3.1, SERVO-3.S; no longer ENC1-2.S, SERVO_MOTOR.P3, U$4.1
- net N$13: now also U6T1.B, U6T1.C, U6T2.B; no longer U6G$1.B, U6G$1.C, U6G$2.B
- net N$16: now also U12.1; no longer U$3.1
- net N$2: now also U6T2.C; no longer U6G$2.C
- net N$3: now also U12.2; no longer U$3.2
- net OUT1: now also J4.P1; no longer MOTOR_CONN1.P1
- net OUT2: now also J4.P2; no longer MOTOR_CONN1.P2
- net OUT3: now also J4.P3; no longer MOTOR_CONN1.P3
- net RPIRESET: now also U5.A4; no longer C22.2, R48.1, U$4.2, U9./RESET
- net VOUT: now also U6T1.E; no longer U6G$1.E
Other:
- note removed: "5V Voltage Regulator and Backpower Protection"
- note removed: "Motor Controller"
- note removed: "Raspberry Pi GPIO"
- note removed: "Raspberry Pi Hat EEPROM"
- moved on the sheet: BATT1, C1, C10, C11, C12, C13, C14, C15, C16, C17, C18, C19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

Commit message: backup
Parts:
- added C30, C31, C32, C39: 0.1u, resistor:C-USC1206
- added H1, H2, H3, H4: MOUNT-HOLE2.8, holes:MOUNT-HOLE2.8
Connections:
- net +5V: now also C30.1, C31.1, C32.1, C39.1
- net GND: now also C30.2, C31.2, C32.2, C39.2
Other:
- moved on the sheet: C38, R45, R46
Changed lines of the file:
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@@
 <part name="GND4" library="supply1" deviceset="GND" device=""/>
 <part name="U8" library="rpibout" deviceset="IPD90P03P4L-04" device=""/>
+<part name="C30" library="resistor" deviceset="C-US" device="C1206" value="0.1u"/>
+<part name="C31" library="resistor" deviceset="C-US" device="C1206" value="0.1u"/>
+<part name="C32" library="resistor" deviceset="C-US" device="C1206" value="0.1u"/>
+<part name="C39" library="resistor" deviceset="C-US" device="C1206" value="0.1u"/>
+<part name="P+19" library="supply1" deviceset="+5V" device=""/>
+<part name="GND6" library="supply1" deviceset="GND" device=""/>
+<part name="H1" library="holes" deviceset="MOUNT-HOLE" device="2.8"/>
+<part name="H2" library="holes" deviceset="MOUNT-HOLE" device="2.8"/>
+<part name="H3" library="holes" deviceset="MOUNT-HOLE" device="2.8"/>
+<part name="H4" library="holes" deviceset="MOUNT-HOLE" device="2.8"/>
 </parts>
 <sheets>
@@
 <instance part="P+18" gate="1" x="73.66" y="180.34"/>
 <instance part="+3V3" gate="G$1" x="45.72" y="180.34"/>
-<instance part="R45" gate="G$1" x="71.12" y="231.14" rot="R90"/>
-<instance part="+3V4" gate="G$1" x="71.12" y="243.84"/>
-<instance part="R46" gate="G$1" x="78.74" y="231.14" rot="R90"/>
+<instance part="R45" gate="G$1" x="76.2" y="231.14" smashed="yes" rot="R90">
+<attribute name="NAME" x="77.2414" y="234.188" size="1.778" layer="95"/>
+<attribute name="VALUE" x="77.47" y="229.108" size="1.778" layer="96"/>
+</instance>
+<instance part="+3V4" gate="G$1" x="63.5" y="243.84"/>
+<instance part="R46" gate="G$1" x="83.82" y="231.14" smashed="yes" rot="R90">
+<attribute name="NAME" x="85.3694" y="234.188" size="1.778" layer="95"/>
+<attribute name="VALUE" x="85.344" y="228.6" size="1.778" layer="96"/>
+</instance>
 <instance part="GND54" gate="1" x="33.02" y="213.36"/>
 <instance part="R47" gate="G$1" x="27.94" y="226.06" rot="R90"/>
 <instance part="+3V6" gate="G$1" x="27.94" y="236.22"/>
-<instance part="C38" gate="G$1" x="86.36" y="231.14"/>
+<instance part="C38" gate="G$1" x="68.58" y="233.68"/>
 <instance part="GND55" gate="1" x="22.86" y="210.82"/>
 <instance part="U9" gate="G$1" x="175.26" y="187.96"/>
@@
 <instance part="J1" gate="G$1" x="17.78" y="215.9" rot="MR0"/>
 <instance part="GND28" gate="1" x="63.5" y="213.36"/>
-<instance part="GND29" gate="1" x="86.36" y="213.36"/>
+<instance part="GND29" gate="1" x="68.58" y="226.06"/>
 <instance part="GND30" gate="1" x="304.8" y="170.18"/>
 <instance part="P+10" gate="1" x="287.02" y="172.72"/>
@@
 <attribute name="VALUE" x="48.26" y="44.958" size="1.778" layer="96" rot="MR180"/>
 </instance>
+<instance part="C30" gate="G$1" x="157.48" y="243.84"/>
+<instance part="C31" gate="G$1" x="165.1" y="243.84"/>
+<instance part="C32" gate="G$1" x="172.72" y="243.84"/>
+<instance part="C39" gate="G$1" x="180.34" y="243.84"/>
+<instance part="P+19" gate="1" x="157.48" y="248.92"/>
+<instance part="GND6" gate="1" x="157.48" y="236.22"/>
+<instance part="H1" gate="G$1" x="302.26" y="33.02"/>
+<instance part="H2" gate="G$1" x="314.96" y="33.02"/>
+<instance part="H3" gate="G$1" x="327.66" y="33.02"/>
+<instance part="H4" gate="G$1" x="340.36" y="33.02"/>
 </instances>
 <busses>
@@
 <pinref part="C38" gate="G$1" pin="2"/>
 <pinref part="GND29" gate="1" pin="GND"/>
-<wire x1="86.36" y1="226.06" x2="86.36" y2="215.9" width="0.1524" layer="91"/>
 </segment>
 <segment>
@@
 <wire x1="360.68" y1="50.8" x2="360.68" y2="48.26" width="0.1524" layer="91"/>
 <junction x="360.68" y="48.26"/>
+</segment>
+<segment>
+<pinref part="GND6" gate="1" pin="GND"/>
+<pinref part="C30" gate="G$1" pin="2"/>
+<pinref part="C39" gate="G$1" pin="2"/>
+<pinref part="C32" gate="G$1" pin="2"/>
+<wire x1="180.34" y1="238.76" x2="172.72" y2="238.76" width="0.1524" layer="91"/>
+<pinref part="C31" gate="G$1" pin="2"/>
+<wire x1="172.72" y1="238.76" x2="165.1" y2="238.76" width="0.1524" layer="91"/>
+<junction x="172.72" y="238.76"/>
+<wire x1="165.1" y1="238.76" x2="157.48" y2="238.76" width="0.1524" layer="91"/>
+<junction x="165.1" y="238.76"/>
+<junction x="157.48" y="238.76"/>
 </segment>
 </net>
@@
 <junction x="360.68" y="60.96"/>
 </segment>
+<segment>
+<pinref part="P+19" gate="1" pin="+5V"/>
+<pinref part="C30" gate="G$1" pin="1"/>
+<pinref part="C31" gate="G$1" pin="1"/>
+<wire x1="157.48" y1="246.38" x2="165.1" y2="246.38" width="0.1524" layer="91"/>
+<junction x="157.48" y="246.38"/>
+<pinref part="C32" gate="G$1" pin="1"/>
+<wire x1="165.1" y1="246.38" x2="172.72" y2="246.38" width="0.1524" layer="91"/>
+<junction x="165.1" y="246.38"/>
+<pinref part="C39" gate="G$1" pin="1"/>
+<wire x1="172.72" y1="246.38" x2="180.34" y2="246.38" width="0.1524" layer="91"/>
+<junction x="172.72" y="246.38"/>
+</segment>
 </net>
 <net name="+3V3" class="0">
@@
 </segment>
 <segment>
-<pinref part="+3V4" gate="G$1" pin="+3V3"/>
-<pinref part="R45" gate="G$1" pin="2"/>
-<wire x1="71.12" y1="241.3" x2="71.12" y2="238.76" width="0.1524" layer="91"/>
-<wire x1="71.12" y1="238.76" x2="71.12" y2="236.22" width="0.1524" layer="91"/>
-<wire x1="71.12" y1="238.76" x2="63.5" y2="238.76" width="0.1524" layer="91"/>
-<junction x="71.12" y="238.76"/>
-<wire x1="63.5" y1="238.76" x2="63.5" y2="226.06" width="0.1524" layer="91"/>
-<pinref part="U4" gate="G$1" pin="VCC"/>
-<wire x1="63.5" y1="226.06" x2="60.96" y2="226.06" width="0.1524" layer="91"/>
-<wire x1="71.12" y1="238.76" x2="78.74" y2="238.76" width="0.1524" layer="91"/>
-<pinref part="R46" gate="G$1" pin="2"/>
-<wire x1="78.74" y1="238.76" x2="78.74" y2="236.22" width="0.1524" layer="91"/>
-<pinref part="C38" gate="G$1" pin="1"/>
-<wire x1="78.74" y1="238.76" x2="86.36" y2="238.76" width="0.1524" layer="91"/>
-<wire x1="86.36" y1="238.76" x2="86.36" y2="233.68" width="0.1524" layer="91"/>
-<junction x="78.74" y="238.76"/>
-</segment>
-<segment>
 <pinref part="R47" gate="G$1" pin="2"/>
 <pinref part="+3V6" gate="G$1" pin="+3V3"/>
@@
 <wire x1="360.68" y1="165.1" x2="360.68" y2="162.56" width="0.1524" layer="91"/>
 <junction x="360.68" y="165.1"/>
+</segment>
+<segment>
+<pinref part="R45" gate="G$1" pin="2"/>
+<wire x1="76.2" y1="238.76" x2="76.2" y2="236.22" width="0.1524" layer="91"/>
+<wire x1="76.2" y1="238.76" x2="68.58" y2="238.76" width="0.1524" layer="91"/>
+<junction x="76.2" y="238.76"/>
+<wire x1="68.58" y1="238.76" x2="63.5" y2="238.76" width="0.1524" layer="91"/>
+<wire x1="63.5" y1="238.76" x2="63.5" y2="226.06" width="0.1524" layer="91"/>
+<pinref part="U4" gate="G$1" pin="VCC"/>
+<wire x1="63.5" y1="226.06" x2="60.96" y2="226.06" width="0.1524" layer="91"/>
+<wire x1="76.2" y1="238.76" x2="83.82" y2="238.76" width="0.1524" layer="91"/>
+<pinref part="R46" gate="G$1" pin="2"/>
+<wire x1="83.82" y1="238.76" x2="83.82" y2="236.22" width="0.1524" layer="91"/>
+<pinref part="+3V4" gate="G$1" pin="+3V3"/>
+<wire x1="63.5" y1="238.76" x2="63.5" y2="241.3" width="0.1524" layer="91"/>
+<junction x="63.5" y="238.76"/>
+<pinref part="C38" gate="G$1" pin="1"/>
+<wire x1="68.58" y1="236.22" x2="68.58" y2="238.76" width="0.1524" layer="91"/>
+<junction x="68.58" y="238.76"/>
 </segment>
 </net>
@@
 <segment>
 <pinref part="R45" gate="G$1" pin="1"/>
-<wire x1="71.12" y1="226.06" x2="71.12" y2="223.52" width="0.1524" layer="91"/>
+<wire x1="76.2" y1="226.06" x2="76.2" y2="223.52" width="0.1524" layer="91"/>
 <label x="33.02" y="142.24" size="1.778" layer="95"/>
 <pinref part="U4" gate="G$1" pin="SDA"/>
-<wire x1="71.12" y1="223.52" x2="60.96" y2="223.52" width="0.1524" layer="91"/>
-<label x="60.96" y="223.52" size="1.778" layer="95"/>
+<wire x1="76.2" y1="223.52" x2="60.96" y2="223.52" width="0.1524" layer="91"/>
+<label x="86.36" y="223.52" size="1.778" layer="95"/>
+<wire x1="93.98" y1="223.52" x2="76.2" y2="223.52" width="0.1524" layer="91"/>
+<junction x="76.2" y="223.52"/>
 </segment>
 <segment>
@@
 <wire x1="337.82" y1="193.04" x2="335.28" y2="193.04" width="0.1524" layer="91"/>
 <pinref part="R27" gate="G$1" pin="1"/>
-<wire x1="335.28" y1="193.04" x2="317.5" y2="193.04" width="0.1524" layer="91"/>
+<wire x1="335.28" y1="193.04" x2="325.12" y2="193.04" width="0.1524" layer="91"/>
 <wire x1="335.28" y1="198.12" x2="335.28" y2="193.04" width="0.1524" layer="91"/>
 <junction x="335.28" y="193.04"/>
-<label x="320.04" y="193.04" size="1.778" layer="95"/>
+<label x="325.12" y="193.04" size="1.778" layer="95"/>
 </segment>
 </net>
@@
 <wire x1="337.82" y1="195.58" x2="330.2" y2="195.58" width="0.1524" layer="91"/>
 <pinref part="R26" gate="G$1" pin="1"/>
-<wire x1="330.2" y1="195.58" x2="317.5" y2="195.58" width="0.1524" layer="91"/>
+<wire x1="330.2" y1="195.58" x2="325.12" y2="195.58" width="0.1524" layer="91"/>
 <wire x1="330.2" y1="198.12" x2="330.2" y2="195.58" width="0.1524" layer="91"/>
 <junction x="330.2" y="195.58"/>
-<label x="320.04" y="195.58" size="1.778" layer="95"/>
+<label x="325.12" y="195.58" size="1.778" layer="95"/>
 </segment>
 </net>
@@
 <segment>
 <pinref part="R46" gate="G$1" pin="1"/>
-<wire x1="78.74" y1="226.06" x2="78.74" y2="220.98" width="0.1524" layer="91"/>
+<wire x1="83.82" y1="226.06" x2="83.82" y2="220.98" width="0.1524" layer="91"/>
 <pinref part="U4" gate="G$1" pin="SCL"/>
-<wire x1="78.74" y1="220.98" x2="60.96" y2="220.98" width="0.1524" layer="91"/>
-<label x="60.96" y="220.98" size="1.778" layer="95"/>
-</segment>
-</net>
+<wire x1="83.82" y1="220.98" x2="60.96" y2="220.98" width="0.1524" layer="91"/>
+<label x="86.36" y="220.98" size="1.778" layer="95"/>
+<wire x1="93.98" y1="220.98" x2="83.82" y2="220.98" width="0.1524" layer="91"/>
+<junction x="83.82" y="220.98"/>
+</segment>
+</net>

Commit message: backup
Parts:
- C16: value 1000uF -> 1000u; device rpibout:CAPACITOR_SMD_J16 -> resistor:CPOL-USE5-10.5
- renumbered BATT1 to BATT, J4 to MOTOR
Connections:
- net ATMEGARESET: now also U9.!RESET!; no longer U9./RESET
- net D12: now also U9.PD6(T1/ADC9/!OC4D!); no longer U9.PD6(T1/ADC9/!OC4D)
- net D5: now also U9.PC6(OC3A/!OC4A!); no longer U9.PC6(OC3A/!OC4A)
- net D9: now also U9.PB5(OC1A/ADC12/!OC4B!); no longer U9.PB5(OC1A/ADC12/!OC4B)
- net GND: now also U9.PE2(!HWB!); no longer U9.PE2(!HWB)
Other:
- note removed: "Motor Backpower Protection"
- note removed: "USB POWER PORT???"
- moved on the sheet: C16, R36, U7
