File: hw/motorcontrol/motorcontrol.sch (EAGLE design)
At the start: 100 parts, among them J3 SWITCH, U1 BTN8982TA, U10 BSS138BKS, U11 DMG2305UX, U12 CRYSTAL, U2 BTN8982TA, U3 BTN8982TA, U4 CAT24C32WI-GT3, U5 ADG3304, U6 MMDT5401, U7 PTR08060W, U8 IPD90P03P4L-04, U9 ATMEGA32U4

Commit message: backup
Parts:
- C1, C10, C12, C3, C6, C7: value 100n -> 0.1u
- C25, C26, C27, C28, C29, C33: value 1u -> 0.1u
- R39, R40, R41: value 750 -> 10k
Connections:
- net +5V: no longer U9.VBUS
- net OUT2: no longer U2.OUT1
- net OUT3: no longer U3.OUT1
Other:
- moved on the sheet: H1, H2, H3, H4

Commit message: backup
Parts:
- C17: value 100n -> 0.1u
Connections:
- removed net N$16: C18.1, R13.1, U12.1, U9.XTAL2
- new net N$7: C19.1, R13.2, U12.1, U9.XTAL1
- net GND: now also U12.2
- net N$3: now also C18.1, R13.1, U12.3, U9.XTAL2; no longer C19.1, R13.2, U12.2, U9.XTAL1
- net OUT2: now also U2.OUT1
- net OUT3: now also U3.OUT1
Other:
- moved on the sheet: R13
Changed lines of the file:
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@@
 <part name="GND17" library="supply1" deviceset="GND" device=""/>
 <part name="D1" library="diode" deviceset="ZENER-DIODE" device="SOD80C" value="10V"/>
-<part name="C17" library="resistor" deviceset="C-US" device="C1206" value="100n"/>
+<part name="C17" library="resistor" deviceset="C-US" device="C1206" value="0.1u"/>
 <part name="GND18" library="supply1" deviceset="GND" device=""/>
 <part name="ENCODER" library="con-molex" deviceset="22-23-2041" device=""/>
@@
 <part name="GND22" library="supply1" deviceset="GND" device=""/>
 <part name="GND23" library="supply1" deviceset="GND" device=""/>
-<part name="U12" library="rpibout" deviceset="CRYSTAL" device=""/>
 <part name="R13" library="resistor" deviceset="R-US_" device="R1206" value="1M"/>
 <part name="P+7" library="supply1" deviceset="+5V" device=""/>
@@
 <part name="U7" library="rpibout" deviceset="PTR08060W" device=""/>
 <part name="C16" library="resistor" deviceset="CPOL-US" device="E5-10.5" value="1000u"/>
+<part name="U12" library="rpibout" deviceset="CRYSTAL" device=""/>
 </parts>
 <sheets>
@@
 <instance part="GND22" gate="1" x="134.62" y="182.88"/>
 <instance part="GND23" gate="1" x="124.46" y="187.96"/>
-<instance part="U12" gate="G$1" x="139.7" y="175.26" smashed="yes" rot="R90">
-<attribute name="NAME" x="143.51" y="171.958" size="1.778" layer="95" font="vector" align="bottom-center"/>
-<attribute name="VALUE" x="146.304" y="177.038" size="1.778" layer="96" font="vector" rot="R180" align="top-center"/>
-</instance>
-<instance part="R13" gate="G$1" x="129.54" y="175.26" smashed="yes" rot="R90">
-<attribute name="NAME" x="131.3434" y="176.53" size="1.778" layer="95"/>
-<attribute name="VALUE" x="131.318" y="172.974" size="1.778" layer="96"/>
+<instance part="R13" gate="G$1" x="142.24" y="175.26" smashed="yes" rot="R90">
+<attribute name="NAME" x="144.0434" y="176.53" size="1.778" layer="95"/>
+<attribute name="VALUE" x="144.018" y="172.974" size="1.778" layer="96"/>
 </instance>
 <instance part="P+7" gate="1" x="259.08" y="241.3"/>
@@
 <instance part="U7" gate="G$1" x="63.5" y="83.82"/>
 <instance part="C16" gate="G$1" x="81.28" y="35.56"/>
+<instance part="U12" gate="G$1" x="129.54" y="175.26" rot="R270"/>
 </instances>
 <busses>
@@
 <pinref part="C19" gate="G$1" pin="2"/>
 <wire x1="116.84" y1="180.34" x2="114.3" y2="180.34" width="0.1524" layer="91"/>
-<wire x1="114.3" y1="180.34" x2="114.3" y2="170.18" width="0.1524" layer="91"/>
+<wire x1="114.3" y1="180.34" x2="114.3" y2="175.26" width="0.1524" layer="91"/>
 <pinref part="GND21" gate="1" pin="GND"/>
 <pinref part="C18" gate="G$1" pin="2"/>
+<wire x1="114.3" y1="175.26" x2="114.3" y2="170.18" width="0.1524" layer="91"/>
 <wire x1="114.3" y1="170.18" x2="114.3" y2="167.64" width="0.1524" layer="91"/>
 <wire x1="116.84" y1="170.18" x2="114.3" y2="170.18" width="0.1524" layer="91"/>
 <junction x="114.3" y="170.18"/>
+<pinref part="U12" gate="G$1" pin="2"/>
+<wire x1="127" y1="175.26" x2="114.3" y2="175.26" width="0.1524" layer="91"/>
+<junction x="114.3" y="175.26"/>
 </segment>
 <segment>
@@
 <pinref part="C11" gate="G$1" pin="2"/>
 <pinref part="C8" gate="G$1" pin="1"/>
-<wire x1="251.46" y1="78.74" x2="259.08" y2="78.74" width="0.1524" layer="91"/>
+<wire x1="251.46" y1="78.74" x2="254" y2="78.74" width="0.1524" layer="91"/>
 <junction x="259.08" y="78.74"/>
+<wire x1="254" y1="78.74" x2="259.08" y2="78.74" width="0.1524" layer="91"/>
 <wire x1="259.08" y1="78.74" x2="271.78" y2="78.74" width="0.1524" layer="91"/>
 <junction x="259.08" y="78.74"/>
 <label x="269.24" y="78.74" size="1.778" layer="95"/>
 <pinref part="U2" gate="G$1" pin="OUT2"/>
+<pinref part="U2" gate="G$1" pin="OUT1"/>
+<wire x1="251.46" y1="81.28" x2="254" y2="81.28" width="0.1524" layer="91"/>
+<wire x1="254" y1="81.28" x2="254" y2="78.74" width="0.1524" layer="91"/>
+<junction x="254" y="78.74"/>
 </segment>
 <segment>
@@
 <pinref part="C15" gate="G$1" pin="2"/>
 <pinref part="C14" gate="G$1" pin="1"/>
-<wire x1="251.46" y1="43.18" x2="259.08" y2="43.18" width="0.1524" layer="91"/>
+<wire x1="251.46" y1="43.18" x2="254" y2="43.18" width="0.1524" layer="91"/>
 <junction x="259.08" y="43.18"/>
+<wire x1="254" y1="43.18" x2="259.08" y2="43.18" width="0.1524" layer="91"/>
 <wire x1="259.08" y1="43.18" x2="271.78" y2="43.18" width="0.1524" layer="91"/>
 <junction x="259.08" y="43.18"/>
 <label x="269.24" y="43.18" size="1.778" layer="95"/>
 <pinref part="U3" gate="G$1" pin="OUT2"/>
+<pinref part="U3" gate="G$1" pin="OUT1"/>
+<wire x1="251.46" y1="45.72" x2="254" y2="45.72" width="0.1524" layer="91"/>
+<wire x1="254" y1="45.72" x2="254" y2="43.18" width="0.1524" layer="91"/>
+<junction x="254" y="43.18"/>
 </segment>
 <segment>
@@
 </segment>
 </net>
-<net name="N$3" class="0">
-<segment>
-<pinref part="U9" gate="G$1" pin="XTAL1"/>
-<pinref part="C19" gate="G$1" pin="1"/>
-<wire x1="149.86" y1="180.34" x2="139.7" y2="180.34" width="0.1524" layer="91"/>
-<pinref part="U12" gate="G$1" pin="2"/>
-<wire x1="139.7" y1="180.34" x2="129.54" y2="180.34" width="0.1524" layer="91"/>
-<wire x1="129.54" y1="180.34" x2="124.46" y2="180.34" width="0.1524" layer="91"/>
-<wire x1="139.7" y1="177.8" x2="139.7" y2="180.34" width="0.1524" layer="91"/>
-<junction x="139.7" y="180.34"/>
-<pinref part="R13" gate="G$1" pin="2"/>
-<junction x="129.54" y="180.34"/>
-</segment>
-</net>
 <net name="N$19" class="0">
 <segment>
@@
 <pinref part="C21" gate="G$1" pin="1"/>
 <wire x1="149.86" y1="190.5" x2="134.62" y2="190.5" width="0.1524" layer="91"/>
-</segment>
-</net>
-<net name="N$16" class="0">
-<segment>
-<pinref part="C18" gate="G$1" pin="1"/>
-<pinref part="R13" gate="G$1" pin="1"/>
-<wire x1="124.46" y1="170.18" x2="129.54" y2="170.18" width="0.1524" layer="91"/>
-<wire x1="129.54" y1="170.18" x2="139.7" y2="170.18" width="0.1524" layer="91"/>
-<junction x="129.54" y="170.18"/>
-<pinref part="U12" gate="G$1" pin="1"/>
-<wire x1="139.7" y1="170.18" x2="139.7" y2="172.72" width="0.1524" layer="91"/>
-<wire x1="139.7" y1="170.18" x2="147.32" y2="170.18" width="0.1524" layer="91"/>
-<junction x="139.7" y="170.18"/>
-<wire x1="147.32" y1="170.18" x2="147.32" y2="172.72" width="0.1524" layer="91"/>
-<pinref part="U9" gate="G$1" pin="XTAL2"/>
-<wire x1="147.32" y1="172.72" x2="149.86" y2="172.72" width="0.1524" layer="91"/>
 </segment>
 </net>
@@
 </segment>
 </net>
+<net name="N$7" class="0">
+<segment>
+<pinref part="U9" gate="G$1" pin="XTAL1"/>
+<pinref part="U12" gate="G$1" pin="1"/>
+<wire x1="129.54" y1="180.34" x2="142.24" y2="180.34" width="0.1524" layer="91"/>
+<wire x1="142.24" y1="180.34" x2="149.86" y2="180.34" width="0.1524" layer="91"/>
+<wire x1="129.54" y1="177.8" x2="129.54" y2="180.34" width="0.1524" layer="91"/>
+<pinref part="C19" gate="G$1" pin="1"/>
+<wire x1="124.46" y1="180.34" x2="129.54" y2="180.34" width="0.1524" layer="91"/>
+<junction x="129.54" y="180.34"/>
+<pinref part="R13" gate="G$1" pin="2"/>
+<junction x="142.24" y="180.34"/>
+</segment>
+</net>
+<net name="N$3" class="0">
+<segment>
+<pinref part="U9" gate="G$1" pin="XTAL2"/>
+<wire x1="147.32" y1="172.72" x2="149.86" y2="172.72" width="0.1524" layer="91"/>
+<wire x1="147.32" y1="170.18" x2="147.32" y2="172.72" width="0.1524" layer="91"/>
+<wire x1="147.32" y1="170.18" x2="142.24" y2="170.18" width="0.1524" layer="91"/>
+<pinref part="U12" gate="G$1" pin="3"/>
+<wire x1="142.24" y1="170.18" x2="129.54" y2="170.18" width="0.1524" layer="91"/>
+<wire x1="129.54" y1="172.72" x2="129.54" y2="170.18" width="0.1524" layer="91"/>
+<pinref part="C18" gate="G$1" pin="1"/>
+<wire x1="124.46" y1="170.18" x2="129.54" y2="170.18" width="0.1524" layer="91"/>
+<junction x="129.54" y="170.18"/>
+<pinref part="R13" gate="G$1" pin="1"/>
+<junction x="142.24" y="170.18"/>
+</segment>
+</net>

Commit message: backup
Parts:
- D2: value 33V -> SMAZX; device diode:DIODE-MELF-MLL41 -> rpibout:SMAZX
Changed lines of the file:
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@@
 <part name="C14" library="resistor" deviceset="C-US" device="C1206" value="220n"/>
 <part name="C15" library="resistor" deviceset="C-US" device="C1206" value="220n"/>
-<part name="D2" library="diode" deviceset="DIODE-" device="MELF-MLL41" value="33V"/>
 <part name="GND19" library="supply1" deviceset="GND" device=""/>
 <part name="GND20" library="supply1" deviceset="GND" device=""/>
@@
 <part name="C16" library="resistor" deviceset="CPOL-US" device="E5-10.5" value="1000u"/>
 <part name="U12" library="rpibout" deviceset="CRYSTAL" device=""/>
+<part name="D2" library="rpibout" deviceset="SMAZX" device=""/>
 </parts>
 <sheets>
@@
 <instance part="C14" gate="G$1" x="259.08" y="40.64"/>
 <instance part="C15" gate="G$1" x="259.08" y="48.26"/>
-<instance part="D2" gate="G$1" x="71.12" y="33.02" rot="R90"/>
 <instance part="GND19" gate="1" x="71.12" y="25.4"/>
 <instance part="GND20" gate="1" x="81.28" y="25.4"/>
@@
 <instance part="C16" gate="G$1" x="81.28" y="35.56"/>
 <instance part="U12" gate="G$1" x="129.54" y="175.26" rot="R270"/>
+<instance part="D2" gate="G$1" x="71.12" y="33.02" rot="R90"/>
 </instances>
 <busses>
@@
 <segment>
 <pinref part="GND19" gate="1" pin="GND"/>
+<wire x1="71.12" y1="30.48" x2="71.12" y2="27.94" width="0.1524" layer="91"/>
 <pinref part="D2" gate="G$1" pin="A"/>
-<wire x1="71.12" y1="30.48" x2="71.12" y2="27.94" width="0.1524" layer="91"/>
 </segment>
 <segment>
@@
 <pinref part="D1" gate="G$1" pin="C"/>
 <wire x1="55.88" y1="40.64" x2="60.96" y2="40.64" width="0.1524" layer="91"/>
-<pinref part="D2" gate="G$1" pin="C"/>
 <wire x1="60.96" y1="40.64" x2="71.12" y2="40.64" width="0.1524" layer="91"/>
 <wire x1="71.12" y1="40.64" x2="71.12" y2="35.56" width="0.1524" layer="91"/>
@@
 <pinref part="U8" gate="G$1" pin="S"/>
 <pinref part="C16" gate="G$1" pin="+"/>
-</segment>
-<segment>
+<pinref part="D2" gate="G$1" pin="C"/>
+</segment>
+<segment>

Commit message: backup
Parts:
- J3: value SWITCH -> B3U-3000P-B; device rpibout:SWITCH -> rpibout:B3U-3000P-B
Changed lines of the file:
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@@
 <part name="+3V7" library="supply1" deviceset="+3V3" device=""/>
 <part name="P+8" library="supply1" deviceset="+5V" device=""/>
-<part name="J3" library="rpibout" deviceset="SWITCH" device=""/>
 <part name="P+1" library="supply1" deviceset="+5V" device=""/>
 <part name="GND24" library="supply1" deviceset="GND" device=""/>
@@
 <part name="U12" library="rpibout" deviceset="CRYSTAL" device=""/>
 <part name="D2" library="rpibout" deviceset="SMAZX" device=""/>
+<part name="J3" library="rpibout" deviceset="B3U-3000P-B" device=""/>
 </parts>
 <sheets>
@@
 <instance part="+3V7" gate="G$1" x="281.94" y="218.44"/>
 <instance part="P+8" gate="1" x="259.08" y="218.44"/>
-<instance part="J3" gate="G$1" x="121.92" y="218.44" rot="R90"/>
 <instance part="P+1" gate="1" x="121.92" y="246.38"/>
 <instance part="GND24" gate="1" x="121.92" y="208.28"/>
@@
 <instance part="U12" gate="G$1" x="129.54" y="175.26" rot="R270"/>
 <instance part="D2" gate="G$1" x="71.12" y="33.02" rot="R90"/>
+<instance part="J3" gate="G$1" x="121.92" y="218.44" rot="R90"/>
 </instances>
 <busses>
@@
 <segment>
 <pinref part="GND24" gate="1" pin="GND"/>
+<wire x1="121.92" y1="210.82" x2="121.92" y2="213.36" width="0.1524" layer="91"/>
 <pinref part="J3" gate="G$1" pin="1"/>
-<wire x1="121.92" y1="210.82" x2="121.92" y2="213.36" width="0.1524" layer="91"/>
 </segment>
 <segment>
@@
 <wire x1="121.92" y1="228.6" x2="121.92" y2="226.06" width="0.1524" layer="91"/>
 <junction x="121.92" y="226.06"/>
-<pinref part="J3" gate="G$1" pin="2"/>
 <wire x1="121.92" y1="226.06" x2="121.92" y2="223.52" width="0.1524" layer="91"/>
 <label x="124.46" y="226.06" size="1.778" layer="95"/>
-</segment>
-<segment>
+<pinref part="J3" gate="G$1" pin="2"/>
+</segment>
+<segment>

Commit message: backup
Connections:
- net +3V3: now also IMU-3.S; no longer IMU-4.S
- net +5V: now also SERVO-2.S; no longer SERVO-1.S
- net D13: now also SERVO-3.S; no longer SERVO-2.S
- net GND: now also IMU-4.S, SERVO-1.S; no longer IMU-3.S, SERVO-3.S
Other:
- moved on the sheet: IMU-3, IMU-4, SERVO-1, SERVO-2, SERVO-3
Changed lines of the file:
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@@
 </instance>
 <instance part="IMU" gate="-2" x="340.36" y="157.48"/>
-<instance part="IMU" gate="-3" x="365.76" y="152.4"/>
-<instance part="IMU" gate="-4" x="365.76" y="165.1"/>
+<instance part="IMU" gate="-3" x="365.76" y="165.1"/>
+<instance part="IMU" gate="-4" x="365.76" y="152.4"/>
 <instance part="GND40" gate="1" x="360.68" y="147.32"/>
 <instance part="+3V2" gate="G$1" x="360.68" y="170.18"/>
@@
 <instance part="C25" gate="G$1" x="360.68" y="195.58"/>
 <instance part="C26" gate="G$1" x="360.68" y="233.68"/>
-<instance part="SERVO" gate="-1" x="365.76" y="238.76" smashed="yes">
-<attribute name="NAME" x="368.3" y="237.998" size="1.524" layer="95"/>
+<instance part="SERVO" gate="-1" x="365.76" y="226.06" smashed="yes">
+<attribute name="NAME" x="368.3" y="225.298" size="1.524" layer="95"/>
 <attribute name="VALUE" x="362.458" y="245.237" size="1.778" layer="96"/>
 </instance>
-<instance part="SERVO" gate="-2" x="340.36" y="233.68"/>
-<instance part="SERVO" gate="-3" x="365.76" y="226.06"/>
+<instance part="SERVO" gate="-2" x="365.76" y="238.76"/>
+<instance part="SERVO" gate="-3" x="340.36" y="233.68"/>
 <instance part="C27" gate="G$1" x="360.68" y="121.92"/>
 <instance part="P+13" gate="1" x="335.28" y="137.16"/>
@@
 </segment>
 <segment>
-<wire x1="360.68" y1="226.06" x2="360.68" y2="223.52" width="0.1524" layer="91"/>
 <pinref part="GND16" gate="1" pin="GND"/>
-<pinref part="SERVO" gate="-3" pin="S"/>
+<pinref part="C26" gate="G$1" pin="2"/>
+<wire x1="360.68" y1="223.52" x2="360.68" y2="226.06" width="0.1524" layer="91"/>
+<pinref part="SERVO" gate="-1" pin="S"/>
+<wire x1="360.68" y1="226.06" x2="360.68" y2="228.6" width="0.1524" layer="91"/>
 <wire x1="363.22" y1="226.06" x2="360.68" y2="226.06" width="0.1524" layer="91"/>
-<pinref part="C26" gate="G$1" pin="2"/>
-<wire x1="360.68" y1="226.06" x2="360.68" y2="228.6" width="0.1524" layer="91"/>
 <junction x="360.68" y="226.06"/>
 </segment>
@@
 <segment>
 <pinref part="C33" gate="G$1" pin="2"/>
+<pinref part="GND40" gate="1" pin="GND"/>
 <wire x1="360.68" y1="154.94" x2="360.68" y2="152.4" width="0.1524" layer="91"/>
-<pinref part="IMU" gate="-3" pin="S"/>
-<wire x1="360.68" y1="152.4" x2="363.22" y2="152.4" width="0.1524" layer="91"/>
-<pinref part="GND40" gate="1" pin="GND"/>
+<pinref part="IMU" gate="-4" pin="S"/>
 <wire x1="360.68" y1="152.4" x2="360.68" y2="149.86" width="0.1524" layer="91"/>
+<wire x1="363.22" y1="152.4" x2="360.68" y2="152.4" width="0.1524" layer="91"/>
 <junction x="360.68" y="152.4"/>
 </segment>
@@
 <pinref part="C26" gate="G$1" pin="1"/>
 <wire x1="360.68" y1="241.3" x2="360.68" y2="238.76" width="0.1524" layer="91"/>
-<pinref part="SERVO" gate="-1" pin="S"/>
+<pinref part="SERVO" gate="-2" pin="S"/>
 <wire x1="360.68" y1="238.76" x2="360.68" y2="236.22" width="0.1524" layer="91"/>
 <wire x1="363.22" y1="238.76" x2="360.68" y2="238.76" width="0.1524" layer="91"/>
@@
 </segment>
 <segment>
-<pinref part="IMU" gate="-4" pin="S"/>
 <pinref part="+3V2" gate="G$1" pin="+3V3"/>
+<pinref part="C33" gate="G$1" pin="1"/>
+<wire x1="360.68" y1="167.64" x2="360.68" y2="165.1" width="0.1524" layer="91"/>
+<pinref part="IMU" gate="-3" pin="S"/>
+<wire x1="360.68" y1="165.1" x2="360.68" y2="162.56" width="0.1524" layer="91"/>
 <wire x1="363.22" y1="165.1" x2="360.68" y2="165.1" width="0.1524" layer="91"/>
-<wire x1="360.68" y1="165.1" x2="360.68" y2="167.64" width="0.1524" layer="91"/>
-<pinref part="C33" gate="G$1" pin="1"/>
-<wire x1="360.68" y1="165.1" x2="360.68" y2="162.56" width="0.1524" layer="91"/>
 <junction x="360.68" y="165.1"/>
 </segment>
@@
 <wire x1="330.2" y1="233.68" x2="337.82" y2="233.68" width="0.1524" layer="91"/>
 <label x="330.2" y="233.68" size="1.778" layer="95"/>
-<pinref part="SERVO" gate="-2" pin="S"/>
-</segment>
-</net>
+<pinref part="SERVO" gate="-3" pin="S"/>
+</segment>
+</net>

Commit message: backup
Parts:
- BATT: value ULTRAFIT_2CIRC -> ULTRAFIT_2CIRCVCLIP; device rpibout:ULTRAFIT_2CIRC -> rpibout:ULTRAFIT_2CIRCVCLIP
- D2: value SMAZX -> 33V
- MOTOR: value ULTRAFIT_3CIRC -> ULTRAFIT_3CIRCVCLIP; device rpibout:ULTRAFIT_3CIRC -> rpibout:ULTRAFIT_3CIRCVCLIP
- XTAL1: value CRYSTAL -> 16MHz
- renumbered U12 to XTAL1
Connections:
- net OUT1: no longer U1.OUT1, U1.OUT2
- net OUT2: no longer U2.OUT1, U2.OUT2
- net OUT3: no longer U3.OUT1, U3.OUT2
Changed lines of the file:
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@@
 <part name="C35" library="resistor" deviceset="CPOL-US" device="E3.5-8" value="220u"/>
 <part name="C36" library="resistor" deviceset="CPOL-US" device="E3.5-8" value="220u"/>
-<part name="BATT" library="rpibout" deviceset="ULTRAFIT_2CIRC" device=""/>
+<part name="BATT" library="rpibout" deviceset="ULTRAFIT_2CIRC" device="VCLIP"/>
 <part name="GND45" library="supply1" deviceset="GND" device=""/>
 <part name="C37" library="resistor" deviceset="C-US" device="C1206" value="1u"/>
@@
 <part name="U2" library="rpibout" deviceset="BTN8982TA" device=""/>
 <part name="U3" library="rpibout" deviceset="BTN8982TA" device=""/>
-<part name="MOTOR" library="rpibout" deviceset="ULTRAFIT_3CIRC" device=""/>
+<part name="MOTOR" library="rpibout" deviceset="ULTRAFIT_3CIRC" device="VCLIP"/>
 <part name="P+12" library="supply1" deviceset="+5V" device=""/>
 <part name="J2" library="pinhead" deviceset="PINHD-2X20" device=""/>
@@
 <part name="U7" library="rpibout" deviceset="PTR08060W" device=""/>
 <part name="C16" library="resistor" deviceset="CPOL-US" device="E5-10.5" value="1000u"/>
-<part name="U12" library="rpibout" deviceset="CRYSTAL" device=""/>
-<part name="D2" library="rpibout" deviceset="SMAZX" device=""/>
+<part name="XTAL1" library="rpibout" deviceset="CRYSTAL" device="" value="16MHz"/>
+<part name="D2" library="rpibout" deviceset="SMAZX" device="" value="33V"/>
 <part name="J3" library="rpibout" deviceset="B3U-3000P-B" device=""/>
 </parts>
@@
 <instance part="U7" gate="G$1" x="63.5" y="83.82"/>
 <instance part="C16" gate="G$1" x="81.28" y="35.56"/>
-<instance part="U12" gate="G$1" x="129.54" y="175.26" rot="R270"/>
+<instance part="XTAL1" gate="G$1" x="129.54" y="175.26" rot="R270"/>
 <instance part="D2" gate="G$1" x="71.12" y="33.02" rot="R90"/>
 <instance part="J3" gate="G$1" x="121.92" y="218.44" rot="R90"/>
@@
 <wire x1="116.84" y1="170.18" x2="114.3" y2="170.18" width="0.1524" layer="91"/>
 <junction x="114.3" y="170.18"/>
-<pinref part="U12" gate="G$1" pin="2"/>
+<pinref part="XTAL1" gate="G$1" pin="2"/>
 <wire x1="127" y1="175.26" x2="114.3" y2="175.26" width="0.1524" layer="91"/>
 <junction x="114.3" y="175.26"/>
@@
 <pinref part="C13" gate="G$1" pin="2"/>
 <pinref part="C4" gate="G$1" pin="1"/>
-<wire x1="251.46" y1="114.3" x2="254" y2="114.3" width="0.1524" layer="91"/>
 <junction x="259.08" y="114.3"/>
 <wire x1="254" y1="114.3" x2="259.08" y2="114.3" width="0.1524" layer="91"/>
@@
 <junction x="259.08" y="114.3"/>
 <label x="269.24" y="114.3" size="1.778" layer="95"/>
-<pinref part="U1" gate="G$1" pin="OUT2"/>
-<pinref part="U1" gate="G$1" pin="OUT1"/>
-<wire x1="251.46" y1="116.84" x2="254" y2="116.84" width="0.1524" layer="91"/>
-<wire x1="254" y1="116.84" x2="254" y2="114.3" width="0.1524" layer="91"/>
-<junction x="254" y="114.3"/>
 </segment>
 <segment>
@@
 <pinref part="C11" gate="G$1" pin="2"/>
 <pinref part="C8" gate="G$1" pin="1"/>
-<wire x1="251.46" y1="78.74" x2="254" y2="78.74" width="0.1524" layer="91"/>
 <junction x="259.08" y="78.74"/>
 <wire x1="254" y1="78.74" x2="259.08" y2="78.74" width="0.1524" layer="91"/>
@@
 <junction x="259.08" y="78.74"/>
 <label x="269.24" y="78.74" size="1.778" layer="95"/>
-<pinref part="U2" gate="G$1" pin="OUT2"/>
-<pinref part="U2" gate="G$1" pin="OUT1"/>
-<wire x1="251.46" y1="81.28" x2="254" y2="81.28" width="0.1524" layer="91"/>
-<wire x1="254" y1="81.28" x2="254" y2="78.74" width="0.1524" layer="91"/>
-<junction x="254" y="78.74"/>
 </segment>
 <segment>
@@
 <pinref part="C15" gate="G$1" pin="2"/>
 <pinref part="C14" gate="G$1" pin="1"/>
-<wire x1="251.46" y1="43.18" x2="254" y2="43.18" width="0.1524" layer="91"/>
 <junction x="259.08" y="43.18"/>
-<wire x1="254" y1="43.18" x2="259.08" y2="43.18" width="0.1524" layer="91"/>
 <wire x1="259.08" y1="43.18" x2="271.78" y2="43.18" width="0.1524" layer="91"/>
 <junction x="259.08" y="43.18"/>
 <label x="269.24" y="43.18" size="1.778" layer="95"/>
-<pinref part="U3" gate="G$1" pin="OUT2"/>
-<pinref part="U3" gate="G$1" pin="OUT1"/>
-<wire x1="251.46" y1="45.72" x2="254" y2="45.72" width="0.1524" layer="91"/>
-<wire x1="254" y1="45.72" x2="254" y2="43.18" width="0.1524" layer="91"/>
-<junction x="254" y="43.18"/>
 </segment>
 <segment>
@@
 <segment>
 <pinref part="U9" gate="G$1" pin="XTAL1"/>
-<pinref part="U12" gate="G$1" pin="1"/>
+<pinref part="XTAL1" gate="G$1" pin="1"/>
 <wire x1="129.54" y1="180.34" x2="142.24" y2="180.34" width="0.1524" layer="91"/>
 <wire x1="142.24" y1="180.34" x2="149.86" y2="180.34" width="0.1524" layer="91"/>
@@
 <wire x1="147.32" y1="170.18" x2="147.32" y2="172.72" width="0.1524" layer="91"/>
 <wire x1="147.32" y1="170.18" x2="142.24" y2="170.18" width="0.1524" layer="91"/>
-<pinref part="U12" gate="G$1" pin="3"/>
+<pinref part="XTAL1" gate="G$1" pin="3"/>
 <wire x1="142.24" y1="170.18" x2="129.54" y2="170.18" width="0.1524" layer="91"/>
 <wire x1="129.54" y1="172.72" x2="129.54" y2="170.18" width="0.1524" layer="91"/>
