File: hw/motorcontrol/motorcontrol.sch (EAGLE design)
At the start: 100 parts, among them J3 B3U-3000P-B, U1 BTN8982TA, U10 BSS138BKS, U11 DMG2305UX, U2 BTN8982TA, U3 BTN8982TA, U4 CAT24C32WI-GT3, U5 ADG3304, U6 MMDT5401, U7 PTR08060W, U8 IPD90P03P4L-04, U9 ATMEGA32U4

Commit message: backup
Parts:
- removed R47: 1k, resistor:R-US_R1206
- added R16: 3.9k, resistor:R-US_R1206
- added R17, R18: 22, resistor:R-US_R1206
- added S2: A6HF-2DIP, rpibout:A6HF-2DIP
- added U12: BSS138BKS, rpibout:BSS138BKS
- J1: device pinhead:PINHD-1X2 -> rpibout:RPIHEADER_2.54-SMD
- J2: value (none) -> USB-MICROB; device pinhead:PINHD-2X20 -> rpibout:USB-MICROB
- LED1: value (none) -> MSL0201RGB; device led:LEDSMT1206 -> rpibout:MSL0201RGB
- R15: value 10k -> 0.51k
- renumbered J3 to S1
Connections:
- new net N$14: LED1.B, U12T1.D
- new net N$16: J2.D-, R18.1
- new net N$22: LED1.G, U12T2.D
- new net N$23: R18.2, U9.D-
- new net N$24: R17.2, U9.D+
- new net N$25: J2.D+, R17.1
- new net N$8: R16.1, S2P2.1, U9.PE2(!HWB!)
- new net RPILEDB: J1.5, U12T1.G
- new net RPILEDG: J1.3, U12T2.G
- new net VBUS: J2.VCC, U9.VBUS
- net +3V3: now also J1.1, J1.17, R15.2, S2P1.1; no longer J2.1, J2.17, R47.2
- net +5V: now also J1.2, J1.4, R16.2; no longer J2.2, J2.4, R15.2
- net GND: now also J1.14, J1.20, J1.25, J1.30, J1.34, J1.39, J1.6, J1.9, J2.GND, LED1.R, S2P2.2, U12T1.S, U12T2.S; no longer J1.2, J2.14, J2.20, J2.25, J2.30, J2.34, J2.39, J2.6, J2.9, LED1.C, U9.PE2(!HWB!)
- net N$12: now also S2P1.2; no longer J1.1, R47.1
- net OUT1: now also U1.OUT
- net OUT2: now also U2.OUT
- net OUT3: now also U3.OUT
- net RPIMISO: now also J1.21; no longer J2.21
- net RPIMOSI: now also J1.19; no longer J2.19
- net RPIRESET: now also J1.12; no longer J2.12
- net RPIROMSCL: now also J1.28; no longer J2.28
- net RPIROMSDA: now also J1.27; no longer J2.27
- net RPISCK: now also J1.23; no longer J2.23
Other:
- moved on the sheet: R15

Commit message: backup
Parts:
- added C40: 0.1u, resistor:C-USC1206
Connections:
- net GND: now also C40.2
- net VPP: now also C40.1
Other:
- moved on the sheet: C12, C3, C7, MOTOR, U12T1, U12T2
