File: hw/motorcontrol/motorcontrol.brd (EAGLE design)
At the start: 65 x 58 mm, 105 parts, among them J2 USB-MICROB, U1 BTN8982TA, U10 BSS138BKS, U11 DMG2305UX, U12 BSS138BKS, U2 BTN8982TA, U3 BTN8982TA, U4 CAT24C32WI-GT3, U5 ADG3304, U6 MMDT5401, U7 PTR08060W, U8 IPD90P03P4L-04, U9 ATMEGA32U4

Commit message: backup
Parts:
- moved R9 38.6 mm to (40.9, 24.1), turned to 90 degrees
- moved R11 36.1 mm to (43.9, 24.1), turned to 90 degrees
- moved R7 30.8 mm to (43.9, 36.1), turned to 90 degrees
- moved R5 26.7 mm to (40.9, 36.1), turned to 90 degrees
- moved R1 5.18 mm to (40.9, 45.5)
- moved R3 4.60 mm to (43.9, 45.5)
- moved R27 3.59 mm to (8.89, 26.9), turned to 270 degrees
- moved R16 2.55 mm to (11.2, 38.9), flipped to the bottom
- moved R26 1.61 mm to (6.60, 26.9), turned to 270 degrees
Routing:
- net +5V: track 45.6 -> 56.2 mm, vias 14 -> 15
- net N$4: track 0.00 -> 8.92 mm, vias 0 -> 1
- net N$1: track 0.00 -> 7.17 mm, vias 0 -> 1
- net N$9: track 0.00 -> 6.38 mm, vias 0 -> 1
- net N$8: track 0.00 -> 4.68 mm
- net N$6: track 0.00 -> 4.63 mm, vias 0 -> 1
- net N$17: track 2.84 -> 6.38 mm
- net D4: track 0.00 -> 3.51 mm
- net D5: track 0.00 -> 3.40 mm
- net N$15: track 2.84 -> 4.63 mm

Commit message: backup
Parts:
- moved R43 8.67 mm to (17.5, 45.2)
- moved R31 5.09 mm to (11.4, 45.2)
- moved R44 5.09 mm to (9.14, 45.2)
- moved U10 5.09 mm to (14.5, 45.0)
- moved R30 2.79 mm to (19.8, 45.2)
- turned C39 to 90 degrees
Routing:
- net +5V: track 56.2 -> 76.7 mm, vias 15 -> 26
- net IMUSCL: track 0.00 -> 16.8 mm
- net IMUSDA: track 0.00 -> 15.8 mm
- net GND: track 139.4 -> 152.6 mm, vias 31 -> 40
- net ATMEGASCL: track 0.00 -> 5.97 mm
- net +3V3: track 33.9 -> 39.8 mm, vias 1 -> 2
- net ATMEGASDA: track 0.00 -> 5.85 mm

Commit message: all planes set, last commit before autoroute
Parts:
- moved U11 1.85 mm to (35.1, 11.9), turned to 0 degrees
Routing:
- net +5V: vias 26 -> 28
- added copper zone on layer 16, net +3V3
Changed lines of the file:
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@@
 <element name="C9" library="resistor" package="C1206" value="1n" x="34.036" y="23.622" rot="R180"/>
 <element name="D1" library="diode" package="SOD80C" value="10V" x="16.51" y="16.002" rot="R270"/>
-<element name="U11" library="rpibout" package="SOT23-3" value="DMG2305UX" x="34.544" y="10.16" rot="MR270"/>
+<element name="U11" library="rpibout" package="SOT23-3" value="DMG2305UX" x="35.052" y="11.938" rot="MR0"/>
 <element name="ENCODER" library="con-molex" package="22-23-2041" value="22-23-2041" x="5.08" y="31.75">
 <attribute name="MPN" value="22-23-2041" x="5.08" y="31.75" size="1.778" layer="27" display="off"/>
@@
 <vertex x="-0.508" y="-0.508"/>
 </polygon>
-<polygon width="0.4064" layer="16" isolate="0.254" thermals="no">
-<vertex x="34.798" y="9.906"/>
+<polygon width="0.3048" layer="16" isolate="0.254" thermals="no">
+<vertex x="33.528" y="11.43"/>
+<vertex x="35.306" y="11.43"/>
+<vertex x="35.306" y="9.906"/>
 <vertex x="36.322" y="9.906"/>
-<vertex x="36.576" y="10.16"/>
-<vertex x="37.846" y="10.16"/>
-<vertex x="37.846" y="8.128"/>
-<vertex x="36.576" y="8.128"/>
-<vertex x="36.068" y="8.636"/>
-<vertex x="34.798" y="8.636"/>
+<vertex x="36.322" y="8.382"/>
+<vertex x="33.528" y="8.382"/>
 </polygon>
-<via x="36.83" y="9.144" extent="1-16" drill="0.4064"/>
-<via x="36.83" y="9.906" extent="1-16" drill="0.4064"/>
-<via x="37.592" y="9.144" extent="1-16" drill="0.4064"/>
-<via x="37.592" y="9.906" extent="1-16" drill="0.4064"/>
+<via x="35.306" y="9.398" extent="1-16" drill="0.4064"/>
+<via x="33.782" y="9.398" extent="1-16" drill="0.4064"/>
+<via x="35.306" y="8.636" extent="1-16" drill="0.4064"/>
+<via x="34.544" y="9.398" extent="1-16" drill="0.4064"/>
 <wire x1="39.482" y1="10.552" x2="39.482" y2="11.318" width="0.4064" layer="16"/>
 <wire x1="39.482" y1="11.318" x2="39.37" y2="11.43" width="0.4064" layer="16"/>
 <via x="39.37" y="11.43" extent="1-16" drill="0.4064"/>
-<via x="36.83" y="8.382" extent="1-16" drill="0.4064"/>
-<via x="37.592" y="8.382" extent="1-16" drill="0.4064"/>
+<via x="33.782" y="8.636" extent="1-16" drill="0.4064"/>
+<via x="34.544" y="8.636" extent="1-16" drill="0.4064"/>
 <wire x1="63.754" y1="24.13" x2="63.754" y2="20.574" width="0.8128" layer="16"/>
 <wire x1="63.754" y1="20.574" x2="63.754" y2="13.716" width="0.8128" layer="16"/>
@@
 <via x="24.892" y="33.274" extent="1-16" drill="0.4064"/>
 <via x="21.59" y="37.592" extent="1-16" drill="0.4064"/>
+<via x="36.068" y="9.398" extent="1-16" drill="0.4064"/>
+<via x="36.068" y="8.636" extent="1-16" drill="0.4064"/>
 </signal>
 <signal name="+3V3">
@@
 <wire x1="8.89" y1="46.888" x2="9.144" y2="46.634" width="0.6096" layer="1"/>
 <wire x1="9.144" y1="46.634" x2="11.43" y2="46.634" width="0.6096" layer="1"/>
-<wire x1="11.43" y1="46.634" x2="28.702" y2="48.768" width="0" layer="19" extent="1-16"/>
-<wire x1="6.35" y1="38.608" x2="9.144" y2="46.634" width="0" layer="19" extent="1-1"/>
-<wire x1="7.518" y1="9.652" x2="6.22" y2="35.56" width="0" layer="19" extent="1-16"/>
-<wire x1="47.368" y1="13.462" x2="33.021" y2="44.704" width="0" layer="19" extent="16-16"/>
+<polygon width="0.4064" layer="16" rank="5">
+<vertex x="-0.762" y="58.674"/>
+<vertex x="65.786" y="58.674"/>
+<vertex x="65.786" y="-0.762"/>
+<vertex x="-0.762" y="-0.762"/>
+</polygon>
+<wire x1="6.22" y1="35.56" x2="7.518" y2="9.652" width="0" layer="19" extent="1-16"/>
 </signal>
 <signal name="VBATT">
@@
 <contactref element="BATT" pad="1"/>
 <polygon width="0.4064" layer="1" thermals="no">
-<vertex x="18.542" y="14.986"/>
-<vertex x="18.542" y="0.508"/>
-<vertex x="37.846" y="0.508"/>
-<vertex x="37.846" y="6.35"/>
-<vertex x="32.766" y="6.35"/>
-<vertex x="24.13" y="14.986"/>
+<vertex x="17.78" y="16.256"/>
+<vertex x="17.78" y="0.508"/>
+<vertex x="43.688" y="0.508"/>
+<vertex x="43.688" y="16.256"/>
 </polygon>
 </signal>
@@
 <contactref element="U6" pad="3"/>
 <contactref element="R38" pad="2"/>
-<wire x1="35.644" y1="11.11" x2="37.658" y2="11.11" width="0.3048" layer="16"/>
-<wire x1="37.658" y1="11.11" x2="39.482" y2="9.286" width="0.3048" layer="16"/>
 <wire x1="39.482" y1="8.752" x2="39.482" y2="9.286" width="0.3048" layer="16"/>
 <wire x1="39.482" y1="8.752" x2="39.232" y2="8.752" width="0.3048" layer="16"/>
@@
 <wire x1="38.1" y1="7.366" x2="37.998" y2="7.366" width="0.3048" layer="16"/>
 <wire x1="37.998" y1="7.366" x2="37.49" y2="6.858" width="0.3048" layer="16"/>
+<wire x1="36.002" y1="10.734" x2="36.83" y2="9.906" width="0.3048" layer="16"/>
+<wire x1="36.83" y1="9.906" x2="36.83" y2="7.366" width="0.3048" layer="16"/>
+<wire x1="36.83" y1="7.366" x2="37.338" y2="6.858" width="0.3048" layer="16"/>
+<wire x1="37.338" y1="6.858" x2="37.49" y2="6.858" width="0.3048" layer="16"/>
+<wire x1="36.002" y1="10.734" x2="36.002" y2="10.838" width="0.3048" layer="16"/>
 </signal>
 <signal name="VPP">

Commit message: backup
Routing:
- net N$8: track 4.68 -> 120.9 mm, vias 0 -> 1
- net D0: track 5.56 -> 97.2 mm
- net D1: track 2.85 -> 80.3 mm, vias 0 -> 1
- net RPIROMSCL: track 5.45 -> 64.0 mm, vias 0 -> 2
- net ATMEGARESET: track 12.6 -> 69.7 mm, vias 0 -> 3
- net D9: track 0.00 -> 57.0 mm
- net VBUS: track 0.00 -> 50.6 mm, vias 0 -> 2
- net RPIROMSDA: track 3.98 -> 52.9 mm, vias 0 -> 2
- net RPILEDG: track 2.02 -> 46.9 mm, vias 0 -> 1
- net RPILEDB: track 1.09 -> 41.5 mm, vias 0 -> 1
- net D13: track 0.00 -> 37.7 mm
- net N$23: track 0.00 -> 33.8 mm, vias 0 -> 1
- net A3: track 10.1 -> 41.4 mm, vias 0 -> 1
- net N$24: track 0.00 -> 28.2 mm, vias 0 -> 1
- net A2: track 10.1 -> 32.9 mm, vias 0 -> 1
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
Commit message: backup
Parts:
- moved C20 2.70 mm to (25.4, 42.2), turned to 180 degrees
- moved C23 0.80 mm to (29.7, 45.5)
- moved R17 0.25 mm to (9.65, 19.1)
- moved R18 0.25 mm to (7.37, 19.1)
- moved R26 0.25 mm to (6.86, 26.9)
- moved R27 0.25 mm to (9.14, 26.9)
Routing:
- net D7: track 9.52 -> 4.84 mm
- net A2: track 32.9 -> 29.6 mm
- net +3V3: track 46.6 -> 44.5 mm
- net GND: track 172.7 -> 173.8 mm
- net D1: track 80.3 -> 81.2 mm
- net N$19: track 4.01 -> 3.09 mm
- net A3: track 41.4 -> 40.8 mm

Commit message: backup
Routing:
- net D7: track 4.84 -> 57.0 mm, vias 0 -> 4
- net D12: track 10.5 -> 50.9 mm, vias 0 -> 2
- net D10: track 0.00 -> 37.0 mm, vias 0 -> 2
- net A4: track 0.00 -> 34.8 mm, vias 0 -> 4
- net +3V3: track 44.5 -> 78.4 mm, vias 4 -> 6

Commit message: backup
Routing:
- net +3V3: track 78.4 -> 70.4 mm, vias 6 -> 11
Changed lines of the file:
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@@
 <grid distance="10" unitdist="mil" unit="mil" style="dots" multiple="1" display="yes" altdistance="2.5" altunitdist="mil" altunit="mil"/>
 <layers>
-<layer number="1" name="Top" color="4" fill="1" visible="yes" active="yes"/>
-<layer number="2" name="Route2" color="6" fill="1" visible="yes" active="yes"/>
+<layer number="1" name="Top" color="4" fill="1" visible="no" active="yes"/>
+<layer number="2" name="Route2" color="6" fill="1" visible="no" active="yes"/>
 <layer number="3" name="Route3" color="4" fill="3" visible="no" active="no"/>
 <layer number="14" name="Route14" color="1" fill="6" visible="no" active="no"/>
-<layer number="15" name="Route15" color="3" fill="1" visible="yes" active="yes"/>
-<layer number="16" name="Bottom" color="1" fill="1" visible="yes" active="yes"/>
+<layer number="15" name="Route15" color="3" fill="1" visible="no" active="yes"/>
+<layer number="16" name="Bottom" color="1" fill="1" visible="no" active="yes"/>
 <layer number="17" name="Pads" color="2" fill="1" visible="yes" active="yes"/>
 <layer number="18" name="Vias" color="2" fill="1" visible="yes" active="yes"/>
@@
 <wire x1="7.62" y1="9.754" x2="7.62" y2="11.43" width="0.4064" layer="1"/>
 <via x="7.62" y="11.43" extent="1-16" drill="0.4064"/>
-<wire x1="10.414" y1="36.068" x2="7.112" y2="36.068" width="0.4064" layer="15"/>
-<wire x1="10.668" y1="35.814" x2="10.414" y2="36.068" width="0.4064" layer="2"/>
-<wire x1="10.668" y1="11.43" x2="10.668" y2="35.814" width="0.4064" layer="2"/>
-<wire x1="7.62" y1="11.43" x2="10.668" y2="11.43" width="0.4064" layer="15"/>
+<wire x1="10.414" y1="36.068" x2="7.112" y2="36.068" width="0.6096" layer="15"/>
+<wire x1="11.938" y1="34.544" x2="10.414" y2="36.068" width="0.6096" layer="2"/>
+<wire x1="11.938" y1="26.416" x2="11.938" y2="27.178" width="0.6096" layer="2"/>
 <via x="10.414" y="36.068" extent="1-16" drill="0.4064"/>
-<via x="10.668" y="11.43" extent="1-16" drill="0.4064"/>
-<wire x1="7.112" y1="37.846" x2="6.35" y2="38.608" width="0.4064" layer="15"/>
-<wire x1="7.112" y1="36.068" x2="7.112" y2="37.846" width="0.4064" layer="15"/>
-<wire x1="47.368" y1="13.462" x2="33.021" y2="44.704" width="0" layer="19" extent="16-16"/>
+<via x="11.938" y="26.416" extent="1-16" drill="0.4064"/>
+<wire x1="11.938" y1="27.178" x2="11.938" y2="34.544" width="0.6096" layer="2"/>
+<wire x1="7.112" y1="37.846" x2="6.35" y2="38.608" width="0.6096" layer="15"/>
+<wire x1="7.112" y1="36.068" x2="7.112" y2="37.846" width="0.6096" layer="15"/>
+<via x="11.938" y="27.178" extent="1-16" drill="0.4064"/>
+<wire x1="13.462" y1="5.334" x2="14.224" y2="5.334" width="0.6096" layer="16"/>
+<wire x1="14.224" y1="5.334" x2="16.764" y2="5.334" width="0.6096" layer="16"/>
+<wire x1="16.764" y1="5.334" x2="18.288" y2="6.858" width="0.6096" layer="16"/>
+<wire x1="18.288" y1="6.858" x2="21.59" y2="6.858" width="0.6096" layer="16"/>
+<via x="13.462" y="5.334" extent="1-16" drill="0.4064"/>
+<via x="14.224" y="5.334" extent="1-16" drill="0.4064"/>
+<via x="22.352" y="6.858" extent="1-16" drill="0.4064"/>
+<wire x1="21.59" y1="6.858" x2="22.352" y2="6.858" width="0.6096" layer="16"/>
+<via x="21.59" y="6.858" extent="1-16" drill="0.4064"/>
 </signal>
 <signal name="VBATT">
