File: hw/motorcontrol/motorcontrol.brd (EAGLE design)
At the start: 65 x 57.2 mm, 105 parts, among them J2 USB-MICROB, U1 BTN8982TA, U10 BSS138BKS, U11 DMG2305UX, U12 BSS138BKS, U2 BTN8982TA, U3 BTN8982TA, U4 CAT24C32WI-GT3, U5 ADG3304, U6 MMDT5401, U7 PTR08060W, U8 IPD90P03P4L-04, U9 ATMEGA32U4

Commit message: backup
Parts:
- removed C29: 10u, resistor:C1206
- removed R31, R44: 3.9k, resistor:R1206
- removed U10: BSS138BKS, rpibout:SOT363
- R16, R26, R27, R30, R43, R45, R46: value 3.9k -> 10k
- S1: value B3U-3000P-B -> SWITCH-GND; device rpibout:B3U-3000P-B -> rpibout:B3F-312X
- U5: value ADG3304 -> ADG3308; device rpibout:TSSOP14 -> rpibout:TSSOP20
- XTAL1: device rpibout:ABM3B -> rpibout:ABLS7M2
- moved XTAL1 53.0 mm to (74.4, 30.7), flipped to the top, turned to 0 degrees
- moved U5 36.1 mm to (71.1, 44.2), flipped to the top, turned to 0 degrees
- moved S1 18.7 mm to (3.56, -9.40), turned to 0 degrees
Connections:
- removed net D14: U9.8
- removed net N$48: U9.22
- new net ATMEGAPD5: U5.12, U9.22
- new net ATMEGASS: U5.15, U9.8
- new net RPICE0: J1.24, U5.6
- net +3V3: no longer C29.1, R31.2, R44.2
- net +5V: now also U5.10, U5.20; no longer U10.2, U10.5, U5.14, U5.8
- net ATMEGAMISO: now also U5.18; no longer U5.12
- net ATMEGAMOSI: now also U5.19; no longer U5.13
- net ATMEGARESET: now also S1.1, U5.16; no longer S1.2, U5.10
- net ATMEGASCK: now also U5.17; no longer U5.11
- net ATMEGASCL: now also U5.14; no longer U10.1
- net ATMEGASDA: now also U5.13; no longer U10.4
- net GND: now also S1.2, S1.3, S1.4, U5.11; no longer C29.2, S1.1, U5.7, XTAL1.GND2, XTAL1.GND4
- net IMUSCL: now also J1.5, U5.7; no longer R44.1, U10.6
- net IMUSDA: now also J1.3, U5.8; no longer R31.1, U10.3
- net N$3: now also XTAL1.2; no longer XTAL1.P3
- net N$7: now also XTAL1.1; no longer XTAL1.P1
- net RPILEDB: now also J1.10, U5.9; no longer J1.5
- net RPILEDG: now also J1.12; no longer J1.3
- net RPIRESET: now also J1.22; no longer J1.12
Routing:
- net RPIRESET: track 25.6 -> 0.00 mm
- net GND: track 167.9 -> 155.4 mm, vias 53 -> 48
- net +5V: track 76.9 -> 67.5 mm, vias 28 -> 27
- net +3V3: track 66.2 -> 58.4 mm
- net ATMEGARESET: track 70.2 -> 62.5 mm
- net ATMEGASCK: track 15.2 -> 8.67 mm
- net ATMEGASDA: track 22.9 -> 16.4 mm
- net IMUSCL: track 16.8 -> 10.4 mm
- net IMUSDA: track 15.8 -> 9.95 mm
- net ATMEGAMISO: track 14.0 -> 10.3 mm
- net RPILEDG: track 48.1 -> 44.6 mm
- net ATMEGAMOSI: track 13.1 -> 10.0 mm
- net N$3: track 10.8 -> 7.88 mm
- net N$7: track 11.7 -> 9.19 mm
- net ATMEGASCL: track 23.1 -> 21.0 mm
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
Commit message: backup
Parts:
- D1: device diode:SOD80C -> rpibout:SOD123
- moved D2 58.3 mm to (71.1, 25.1), turned to 0 degrees
- moved D1 54.1 mm to (70.4, 21.3), turned to 0 degrees
- moved S1 21.4 mm to (0.00, 11.7), turned to 270 degrees
- moved LED1 10.1 mm to (11.2, 9.65)
- moved R15 9.49 mm to (8.64, 18.8)
- moved R17 5.39 mm to (10.4, 24.4)
- moved R18 5.39 mm to (8.13, 24.4)
- moved U12 4.83 mm to (9.40, 13.2)
- moved J2 4.83 mm to (0.00, 24.1)
Routing:
- net VBUS: track 50.6 -> 12.9 mm, vias 2 -> 1
- net N$23: track 34.3 -> 3.56 mm, vias 1 -> 0
- net RPILEDB: track 40.5 -> 10.4 mm, vias 1 -> 0
- net N$24: track 28.3 -> 7.89 mm, vias 1 -> 0
- net ATMEGARESET: track 62.5 -> 52.2 mm
- net GND: track 155.4 -> 149.2 mm, vias 48 -> 47
- net N$25: track 5.85 -> 0.00 mm
- net RPILEDG: track 44.6 -> 39.3 mm, vias 1 -> 0
- net N$14: track 4.96 -> 0.00 mm
- net N$10: track 4.51 -> 0.00 mm
- net N$16: track 3.20 -> 0.00 mm
- net N$22: track 2.93 -> 0.00 mm
- net N$21: track 11.4 -> 8.47 mm
- net +3V3: track 58.4 -> 56.6 mm, vias 11 -> 8
- net VPP: track 0.65 -> 0.00 mm

Commit message: backup
Parts:
- LED1: value MSL0201RGB -> LED_3COLOR_COMMONA1411; device rpibout:MSL0201RGB -> rpibout:150141M173100
- R15: value 0.51k -> 267
- moved D2 58.2 mm to (13.7, 15.7), turned to 270 degrees
- moved U5 54.8 mm to (16.5, 49.0)
- moved D1 54.1 mm to (16.5, 16.0), turned to 270 degrees
- moved XTAL1 53.1 mm to (21.8, 23.1), flipped to the bottom, turned to 180 degrees
- moved C34 35.7 mm to (70.9, 13.7)
- moved R36 31.5 mm to (70.6, 17.3)
- moved C23 20.9 mm to (9.40, 50.5), flipped to the top, turned to 90 degrees
- moved C24 13.2 mm to (23.4, 51.6), flipped to the top, turned to 0 degrees
- moved LED1 12.0 mm to (2.79, 18.3), turned to 0 degrees
- moved R48 10.3 mm to (6.10, 12.7), flipped to the bottom, turned to 180 degrees
- moved U12 8.13 mm to (9.40, 5.08)
- moved C22 7.71 mm to (6.10, 10.7), flipped to the bottom, turned to 0 degrees
- moved C25 7.11 mm to (2.79, 35.6)
- moved R43 6.84 mm to (23.4, 48.8), turned to 0 degrees
- moved C18 4.13 mm to (26.9, 19.6), turned to 270 degrees
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Connections:
- net GND: now also J2.GND3, J2.GND4
Routing:
- net +3V3: track 56.6 -> 5.94 mm, vias 8 -> 1
- net RPILEDG: track 39.3 -> 0.00 mm
- net ATMEGARESET: track 52.2 -> 13.5 mm, vias 3 -> 1
- net GND: track 149.2 -> 118.5 mm, vias 47 -> 40
- net +5V: track 67.5 -> 44.1 mm, vias 27 -> 24
- net ATMEGASCL: track 21.0 -> 0.00 mm, vias 1 -> 0
- net IMUSCL: track 10.4 -> 0.00 mm
- net RPILEDB: track 10.4 -> 0.00 mm
- net ATMEGAMOSI: track 10.0 -> 0.00 mm
- net IMUSDA: track 9.95 -> 0.00 mm
- net N$7: track 9.19 -> 0.00 mm
- net N$21: track 8.47 -> 0.00 mm
- net N$3: track 7.88 -> 0.00 mm
- net N$15: track 5.80 -> 0.00 mm, vias 1 -> 0
- net RPIMOSI: track 5.00 -> 0.00 mm
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Other:
- board text added: "Pi Car Control Board v2.1 WashU ESE Dept May 2017"
- board text removed: "Pi Car Control Board v2.0 WashU ESE Dept May 2017"

Commit message: new schematic is ready
Parts:
- removed C22: 0.1u, resistor:C1206
- added R19, R20, R21, R22, R23: 10k, resistor:R1206
- added U10: SN74LV4T125, rpibout:TSSOP14
- added U13: BSS138BKS, rpibout:SOT363
- U5: value ADG3308 -> SN74LV4T125; device rpibout:TSSOP20 -> rpibout:TSSOP14
- moved U5 1.37 mm to (16.0, 50.3)
Connections:
- net N$23 renamed ATMEGAD-
- net N$24 renamed ATMEGAD+
- new net RPIGND: J1.25, R22.1, U5.1, U5.10, U5.13, U5.4
- net +3V3: now also R20.2, R21.2, R48.2, U10.14, U13.2, U13.5; no longer S2.P1.1, U5.1
- net +5V: now also R19.2, R22.2, R23.2, U5.14; no longer C22.1, R48.2, U5.10, U5.20
- net ATMEGAMISO: now also U10.2; no longer U5.18
- net ATMEGAMOSI: now also U5.3; no longer U5.19
- net ATMEGAPD5: now also U10.5; no longer U5.12
- net ATMEGARESET: now also R23.1, U5.8; no longer C22.2, R48.1, S1.1, U5.16
- net ATMEGASCK: now also U5.6; no longer U5.17
- net ATMEGASCL: now also U13.6; no longer U5.14
- net ATMEGASDA: now also U13.3; no longer U5.13
- net ATMEGASS: now also U5.11; no longer U5.15
- net GND: now also U10.1, U10.10, U10.12, U10.13, U10.4, U10.7, U10.9, U5.7; no longer J1.25, U5.11
- net IMUSCL: now also R20.1, U13.1; no longer U5.7
- net IMUSDA: now also R21.1, U13.4; no longer U5.8
- net N$12: now also R19.1; no longer S2.P1.2, U4.7
- net RPICE0: now also U5.12; no longer U5.6
- net RPILEDB: now also U10.6; no longer U5.9
- net RPIMISO: now also U10.3; no longer U5.3
- net RPIRESET: now also R48.1, S1.1, U5.9; no longer U5.5
- net RPISCK: now also U5.5; no longer U5.4
Routing:
- net VBUS: track 12.9 -> 0.00 mm, vias 1 -> 0
- net N$18: track 11.5 -> 0.00 mm
- net N$5: track 11.5 -> 0.03 mm
- net N$11: track 11.5 -> 0.03 mm
- net A3: track 40.8 -> 30.7 mm
- net A2: track 29.7 -> 19.6 mm
- net A4: track 34.7 -> 24.8 mm
- net ATMEGAD+: track 7.89 -> 0.00 mm
- net N$12: track 4.92 -> 0.00 mm, vias 1 -> 0
- net ATMEGAD-: track 3.56 -> 0.00 mm
- net +3V3: track 5.94 -> 3.12 mm, vias 1 -> 0
- net GND: track 118.5 -> 116.4 mm, vias 40 -> 39

Commit message: fixed RPi-Arduino buffer for reset pin
Parts:
- removed R19, R23: 10k, resistor:R1206
Connections:
- net +3V3: now also S2.P1.2; no longer R48.2
- net +5V: now also R48.2; no longer R19.2, R23.2
- net ATMEGARESET: now also R48.1, S1.1; no longer R23.1
- net N$12: now also S2.P1.1, U4.7; no longer R19.1
- net RPIRESET: no longer R48.1, S1.1

Commit message: backup
Parts:
- removed C37: 1u, resistor:C1206
- U11: value DMG2305UX -> SI2333CDS-T1-GE3
- moved R36 36.2 mm to (35.3, 9.40)
- moved C34 31.1 mm to (39.9, 16.5), flipped to the bottom
- moved R15 13.2 mm to (8.89, 5.59), turned to 270 degrees
- moved R37 10.9 mm to (30.0, 7.37), turned to 180 degrees
- moved U11 6.76 mm to (40.6, 8.13), turned to 180 degrees
- moved R17 6.59 mm to (8.64, 18.0), turned to 0 degrees
- moved R38 6.48 mm to (30.0, 9.65)
- moved U6 4.58 mm to (35.8, 8.13), turned to 90 degrees
- moved R18 4.10 mm to (8.64, 20.3), turned to 0 degrees
- moved U12 3.78 mm to (11.9, 7.87)
- moved C40 1.61 mm to (40.9, 19.3), turned to 0 degrees
- moved C35 1.55 mm to (29.5, 4.32), turned to 180 degrees
- moved C36 1.27 mm to (39.6, 14.0), turned to 180 degrees
- moved BATT 0.76 mm to (18.5, 2.54)
- moved D2 0.51 mm to (13.2, 15.7)
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Connections:
- net GND: no longer C37.2
- net VOUT: no longer C37.1
Routing:
- net GND: track 116.4 -> 106.2 mm, vias 39 -> 36
- net N$2: track 8.35 -> 0.00 mm
- net N$13: track 5.00 -> 0.65 mm
- net +5V: track 44.1 -> 43.2 mm, vias 24 -> 21

Commit message: backup
Parts:
- moved C23 16.0 mm to (24.6, 55.4), turned to 0 degrees
- moved R20 15.3 mm to (11.2, 51.3), turned to 90 degrees
- moved R15 14.5 mm to (7.62, 20.1), turned to 90 degrees
- moved R43 14.4 mm to (12.7, 39.1), turned to 270 degrees
- moved R21 12.9 mm to (8.13, 51.3), turned to 90 degrees
- moved R22 12.7 mm to (19.1, 55.4)
- moved R30 10.6 mm to (15.7, 38.9), turned to 270 degrees
- moved C24 10.4 mm to (13.7, 55.4), turned to 180 degrees
- moved U10 8.32 mm to (23.4, 48.5), turned to 90 degrees
- moved R18 6.55 mm to (12.4, 25.7)
- moved R17 6.35 mm to (12.4, 23.1)
- moved R48 6.27 mm to (8.38, 6.86), flipped to the top, turned to 270 degrees
- moved U12 5.64 mm to (8.64, 12.4), turned to 270 degrees
- moved C17 3.64 mm to (21.8, 7.62), flipped to the bottom
- moved C34 2.03 mm to (37.8, 16.5)
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Routing:
- net D7: track 57.0 -> 7.97 mm, vias 4 -> 0
- net +3V3: track 3.11 -> 33.2 mm, vias 0 -> 1
- net IMUSCL: track 0.00 -> 13.1 mm
- net N$21: track 0.00 -> 12.3 mm
- net GND: track 106.2 -> 117.7 mm
- net IMUSDA: track 0.00 -> 10.6 mm
- net N$41: track 0.00 -> 10.4 mm
- net N$22: track 0.00 -> 9.90 mm
- net A4: track 24.8 -> 34.7 mm
- net A2: track 19.6 -> 29.0 mm
- net A3: track 30.7 -> 40.0 mm
- net ATMEGARESET: track 13.5 -> 22.5 mm
- net N$14: track 0.00 -> 7.38 mm
- net ATMEGASCL: track 0.00 -> 7.26 mm
- net N$25: track 0.00 -> 6.79 mm
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
Commit message: backup
Parts:
- moved R20 3.05 mm to (8.13, 51.3)
- moved R21 3.05 mm to (11.2, 51.3)
- moved R37 2.96 mm to (28.4, 9.91)
- moved R38 2.75 mm to (28.4, 7.37)
- moved U11 2.54 mm to (38.1, 8.13)
- moved U6 1.93 mm to (34.0, 8.89)
- moved R30 0.57 mm to (15.2, 39.1)
- moved C3 0.52 mm to (42.7, 55.5)
- moved C19 0.36 mm to (17.0, 19.3)
- moved C18 0.36 mm to (26.7, 19.3)
- moved C7 0.13 mm to (42.7, 43.6)
- moved C12 0.13 mm to (42.7, 31.6)
Routing:
- net D13: track 37.8 -> 21.0 mm
- net N$12: track 0.00 -> 12.7 mm, vias 0 -> 1
- net IMUSCL: track 13.1 -> 24.4 mm, vias 0 -> 1
- net ATMEGASDA: track 13.4 -> 24.2 mm, vias 1 -> 3
- net ATMEGAMISO: track 9.67 -> 0.00 mm, vias 1 -> 0
- net ATMEGASCK: track 8.67 -> 0.00 mm, vias 2 -> 0
- net IMUSDA: track 10.6 -> 16.7 mm, vias 0 -> 2
- net +3V3: track 33.2 -> 38.4 mm, vias 1 -> 3
- net +5V: track 48.6 -> 53.4 mm
- net GND: track 117.7 -> 118.0 mm, vias 36 -> 35
