File: hw/motorcontrol/motorcontrol.brd (EAGLE design)
At the start: 65 x 57.2 mm, 104 parts, among them J2 USB-MICROB, U1 BTN8982TA, U10 SN74LV4T125, U11 SI2333CDS-T1-GE3, U12 BSS138BKS, U13 BSS138BKS, U2 BTN8982TA, U3 BTN8982TA, U4 CAT24C32WI-GT3, U5 SN74LV4T125, U6 MMDT5401, U7 PTR08060W, U8 IPD90P03P4L-04, U9 ATMEGA32U4

Commit message: before autoroute
Parts:
- moved C38 10.9 mm to (49.3, 2.54), turned to 0 degrees
- moved C34 3.88 mm to (34.5, 14.5), turned to 90 degrees
- moved C17 0.57 mm to (21.3, 7.37)
- moved R5 0.51 mm to (41.4, 36.1)
- moved R9 0.51 mm to (41.4, 25.1)
- moved U6 0.51 mm to (34.0, 8.38), turned to 270 degrees
- moved C3 0.28 mm to (42.4, 55.4)
- moved R45 0.25 mm to (49.3, 5.84)
- moved R46 0.25 mm to (49.3, 8.13)
- moved C18 0.13 mm to (26.8, 19.3)
- moved C19 0.13 mm to (17.1, 19.3)
- moved R13 0.13 mm to (22.0, 19.3)
- moved XTAL1 0.13 mm to (22.0, 23.1)
Connections:
- net GND: now also J1.25; no longer J1.6
- net RPIGND: now also J1.6; no longer J1.25
Routing:
- net GND: track 118.0 -> 137.5 mm, vias 35 -> 40
- net N$3: track 0.00 -> 14.7 mm
- net N$2: track 0.00 -> 14.5 mm, vias 0 -> 2
- net N$7: track 0.00 -> 14.5 mm
- net N$5: track 2.09 -> 10.5 mm, vias 0 -> 2
- net N$18: track 2.05 -> 9.97 mm, vias 0 -> 2
- net N$11: track 2.09 -> 10.0 mm, vias 0 -> 2
- net N$13: track 0.65 -> 6.58 mm
- net VBATT: track 0.00 -> 4.97 mm
- net N$15: track 0.00 -> 4.51 mm, vias 0 -> 1
- net IMUSDA: track 16.7 -> 18.6 mm
- net D7: track 7.97 -> 6.19 mm
- net +5V: track 53.4 -> 54.6 mm, vias 22 -> 23
- net N$6: track 4.63 -> 5.29 mm
- net D4: track 32.1 -> 32.6 mm
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
Commit message: backup
Routing:
- net RPILEDB: track 0.00 -> 61.8 mm, vias 0 -> 5
- net ATMEGARESET: track 22.3 -> 83.7 mm, vias 1 -> 4
- net D7: track 6.19 -> 60.7 mm, vias 0 -> 2
- net ATMEGASDA: track 24.2 -> 78.2 mm
- net RPILEDG: track 0.00 -> 53.5 mm, vias 0 -> 2
- net VBUS: track 0.00 -> 47.8 mm, vias 0 -> 4
- net ATMEGASS: track 0.00 -> 30.4 mm, vias 0 -> 2
- net ATMEGAMOSI: track 0.00 -> 28.9 mm, vias 0 -> 2
- net ATMEGAPD5: track 0.00 -> 27.2 mm, vias 0 -> 2
- net RPICE0: track 0.00 -> 25.9 mm, vias 0 -> 1
- net RPISCK: track 0.00 -> 25.3 mm, vias 0 -> 2
- net +5V: track 54.6 -> 79.9 mm, vias 23 -> 24
- net RPIGND: track 0.00 -> 24.6 mm, vias 0 -> 1
- net ATMEGASCK: track 0.00 -> 24.2 mm, vias 0 -> 1
- net ATMEGAMISO: track 0.00 -> 23.9 mm, vias 0 -> 1
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
Commit message: backup
Parts:
- removed R16: 10k, resistor:R1206
- added C22, C29: 0.1u, resistor:C1206
- added R19, R23, R24, R25, R28, R32: 267, resistor:R1206
- added R29: 10k, resistor:R1206
- added RCVR: 22-23-2031, con-molex:22-23-2031
- C11, C13, C14, C15, C4, C8: value 220n -> 0.22u
- R12, R4, R8: value 0.51k -> 510
- R22: value 10k -> 267
- moved R22 102.4 mm to (1.02, -45.5)
- moved R46 96.9 mm to (1.02, -75.9), flipped to the top
- moved J1 73.0 mm to (24.6, -20.1)
Connections:
- net ATMEGAMISO renamed ATPB3
- net ATMEGAPD5 renamed ATPD5
- net ATMEGASCL renamed ATSCL
- net ATMEGASDA renamed ATSDA
- net D10 renamed ATOC1B
- net D11 renamed ATOC1C
- net D9 renamed ATOC1A
- removed net A0: U9.36
- removed net A1: U9.37
- removed net A2: C2.1, R2.2, U1.6, U9.38
- removed net A3: C5.1, R6.2, U2.6, U9.39
- removed net A4: C9.1, R10.2, U3.6, U9.40
- removed net A5: U9.41
- removed net ATMEGAMOSI: U5.3, U9.10
- removed net ATMEGARESET: R48.1, S1.1, U5.8, U9.13
- removed net ATMEGASCK: U5.6, U9.9
- removed net ATMEGASS: U5.11, U9.8
- removed net D0: HALL1.3, R39.1, U9.20
- removed net D1: HALL2.3, R40.1, U9.21
- removed net D12: R5.1, U9.26
- removed net D13: SERVO.3, U9.32
- removed net D4: R9.1, U9.25
- removed net D5: ENCODER.4, R27.1, U9.31
- removed net D6: R1.1, U9.27
- removed net D7: HALL3.3, R41.1, U9.1
- removed net D8: ENCODER.3, R26.1, U9.28
- removed net N$8: R16.1, S2.P2.1, U9.33
- new net ATADC0: C2.1, R2.2, U1.6, U9.41
- new net ATADC1: C5.1, R6.2, U2.6, U9.40
- new net ATADC2: C9.1, R10.2, U3.6
- new net ATADC4: U9.39
- new net ATHWB: S2.P2.1, U9.33
- new net ATICP3: RCVR.3, U9.32
- new net ATINT6: ENCODER.3, R26.1, U9.1
- new net ATOC3A: SERVO.3, U9.31
- new net ATPB0: HALL1.3, R25.2, R39.1, U9.8
- new net ATPB1: HALL2.3, R24.2, R40.1, U9.9
- new net ATPB2: HALL3.3, R23.2, R41.1, U9.10
- new net ATPB4: ENCODER.4, R27.1, U9.28
- new net ATPD4: U9.25
- new net ATPD6: U9.26
- new net ATPD7: U9.27
- new net ATPF5: R1.1, U9.38
- new net ATPF6: R5.1, U9.37
- new net ATPF7: R9.1, U9.36
- new net ATRESET: C22.1, R19.2, R22.2, R48.1, U9.13
- new net ATRX1: R32.2, U9.20
- new net ATTX1: U10.9, U9.21
- new net N$11: R28.2, U10.6
- new net N$18: R22.1, U5.3
- new net N$23: R19.1, S1.1
- new net N$27: R23.1, U5.6
- new net N$28: R24.1, U5.8
- new net N$31: R32.1, U5.11
- new net RPIRX0: J1.10, U10.8
- new net RPITX0: J1.8, U5.12
- net +5V: now also C29.1, R29.2, RCVR.2; no longer R16.2, R22.2
- net GND: now also C22.2, C29.2, RCVR.1, U7.3; no longer U10.9, U7.P3
- net N$41: now also U7.5; no longer U7.P5
- net RPICE0: now also R25.1; no longer U5.12
- net RPIGND: now also R29.1; no longer R22.1
- net RPILEDB: now also J1.16, R28.1; no longer J1.10, U10.6
- net RPIMOSI: now also U5.5; no longer U5.2
- net RPIRESET: now also U5.2; no longer U5.9
- net RPISCK: now also U5.9; no longer U5.5
- net VBATT: now also U7.2; no longer U7.P2
- net VOUT: now also U7.4; no longer U7.P4
Routing:
- net N$8: track 120.5 -> 0.00 mm, vias 1 -> 0
- net ATHWB: track 0.00 -> 119.9 mm, vias 0 -> 1
- net ATPB0: track 0.00 -> 91.7 mm, vias 0 -> 6
- net ATMEGARESET: track 83.7 -> 0.00 mm, vias 4 -> 0
- net ATRESET: track 0.00 -> 82.8 mm, vias 0 -> 4
- net ATINT6: track 0.00 -> 62.7 mm, vias 0 -> 2
- net D0: track 62.5 -> 0.00 mm, vias 4 -> 0
- net D7: track 60.7 -> 0.00 mm, vias 2 -> 0
- net D1: track 49.0 -> 0.00 mm, vias 4 -> 0
- net ATTX1: track 0.00 -> 48.2 mm, vias 0 -> 4
- net A3: track 39.8 -> 0.00 mm, vias 1 -> 0
- net A4: track 34.7 -> 0.00 mm, vias 4 -> 0
- net D6: track 34.6 -> 0.00 mm, vias 3 -> 0
- net ATPD7: track 0.00 -> 34.5 mm, vias 0 -> 3
- net D12: track 33.4 -> 0.00 mm, vias 2 -> 0
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
Commit message: backup
Parts:
- added C37: 0.1u, resistor:C1206
- added EXTRAIO: 22-23-2041, con-molex:22-23-2041
- added R16: 267, resistor:R1206
- moved RCVR 100.9 mm to (50.5, 10.4), turned to 180 degrees
- moved S2 66.1 mm to (18.5, 59.9)
Connections:
- net ATPB3 renamed ATMISO
- removed net ATHWB: S2.P2.1, U9.33
- removed net ATPD4: U9.25
- new net ATICP1: EXTRAIO.4, U9.25
- new net RPIGPIO4: J1.7, R16.1
- new net U5OE: R16.2, S2.P2.2, U5.1, U5.10, U5.13, U5.4
- net +5V: now also C37.1, EXTRAIO.2
- net ATOC1A: now also EXTRAIO.3
- net GND: now also C37.2, EXTRAIO.1, J1.6, U9.33; no longer J1.14, S2.P2.2
- net RPIGND: now also J1.14, S2.P2.1; no longer J1.6, R29.1, U5.1, U5.10, U5.13, U5.4
Routing:
- net ATHWB: track 119.9 -> 0.00 mm, vias 1 -> 0
- net GND: track 131.9 -> 225.9 mm
- net ATPD4: track 31.4 -> 0.00 mm, vias 5 -> 0
- net ATICP1: track 0.00 -> 31.4 mm, vias 0 -> 5
- net N$12: track 12.7 -> 2.70 mm, vias 1 -> 0
- net +3V3: track 50.8 -> 49.6 mm, vias 4 -> 3

Commit message: backup
Parts:
- removed R32: 267, resistor:R1206
- R16: value 267 -> 10k
- U4: value CAT24C32WI-GT3 -> CAT24C32
- moved R16 152.2 mm to (10.9, 46.0), flipped to the bottom
- moved C37 123.2 mm to (54.4, 7.62), flipped to the bottom, turned to 180 degrees
- moved R46 120.2 mm to (52.3, 32.8), flipped to the bottom
- moved C29 118.5 mm to (2.79, 36.1), flipped to the bottom
- moved R29 115.0 mm to (22.4, 55.4)
- moved R28 95.7 mm to (22.9, 41.7), turned to 90 degrees
- moved R22 90.0 mm to (10.9, 43.9), turned to 180 degrees
- moved R25 77.1 mm to (10.9, 37.1), turned to 180 degrees
- moved R24 73.3 mm to (10.9, 39.4), turned to 180 degrees
- moved J1 73.0 mm to (32.5, 52.5)
- moved R23 69.5 mm to (10.9, 41.7), turned to 180 degrees
- moved RCVR 54.7 mm to (3.81, 38.9), turned to 0 degrees
- moved C38 39.1 mm to (49.3, 41.7), turned to 270 degrees
- moved U4 36.6 mm to (54.6, 41.7), turned to 180 degrees
- moved R45 30.1 mm to (52.3, 35.8)
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Connections:
- net ATMEGAD+ renamed ATD+
- net ATMEGAD- renamed ATD-
- net RPISCK renamed RPISCLK
- net VBUS renamed ATVBUS
- removed net N$31: R32.1, U5.11
- removed net RPIGPIO4: J1.7, R16.1
- removed net RPITX0: J1.8, U5.12
- new net N$29: R25.1, U5.11
- new net N$8: S2.P1.1, U9.33
- net +3V3: no longer S2.P1.2
- net ATOC1A: no longer EXTRAIO.3
- net ATOC1C: now also EXTRAIO.3
- net ATRX1: now also J1.8; no longer R32.2
- net GND: now also R16.2, U4.7; no longer U9.33
- net N$12: now also R16.1, S2.P1.2; no longer S2.P1.1, U4.7
- net N$3: now also C19.1, U9.17; no longer C18.1, U9.16
- net N$7: now also C18.1, U9.16; no longer C19.1, U9.17
- net RPICE0: now also U5.12; no longer R25.1
- net RPIGND: now also U5.1
- net U5OE: now also R29.1; no longer R16.2, U5.1
Routing:
- net GND: track 225.9 -> 100.8 mm, vias 35 -> 33
- net ATPB0: track 91.7 -> 0.00 mm, vias 6 -> 0
- net ATRESET: track 82.8 -> 0.00 mm, vias 4 -> 0
- net ATSDA: track 78.2 -> 0.00 mm, vias 3 -> 0
- net RPIROMSCL: track 63.5 -> 0.00 mm, vias 2 -> 0
- net ATINT6: track 62.7 -> 0.00 mm, vias 2 -> 0
- net RPILEDB: track 61.7 -> 0.00 mm, vias 5 -> 0
- net RPILEDG: track 53.5 -> 0.00 mm, vias 2 -> 0
- net RPIROMSDA: track 51.8 -> 0.00 mm, vias 2 -> 0
- net +5V: track 77.8 -> 27.1 mm, vias 24 -> 18
- net +3V3: track 49.6 -> 0.00 mm, vias 3 -> 0
- net ATTX1: track 48.2 -> 0.00 mm, vias 4 -> 0
- net ATVBUS: track 47.8 -> 0.06 mm, vias 4 -> 0
- net ATPD7: track 34.5 -> 0.00 mm, vias 3 -> 0
- net ATPD6: track 32.8 -> 0.00 mm, vias 2 -> 0
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Other:
- board text removed: "1: EEPROM WP Enable 2: Bootloader Enable"

Commit message: backup
Parts:
- added C41: 0.1u, resistor:C1206
- moved U4 22.5 mm to (51.8, 19.3), turned to 0 degrees
- moved C38 21.6 mm to (55.9, 21.1)
- moved R45 8.03 mm to (54.9, 28.2), turned to 180 degrees
- moved R46 7.31 mm to (54.9, 25.9), turned to 180 degrees
- moved C33 4.83 mm to (2.79, 29.0), turned to 0 degrees
- moved R41 3.14 mm to (51.3, 10.9), turned to 90 degrees
- moved R40 3.09 mm to (53.6, 10.9)
- moved R39 3.06 mm to (55.9, 10.9)
- moved R22 1.37 mm to (11.4, 45.2)
- moved R48 1.27 mm to (9.91, 10.9)
- moved C37 1.27 mm to (54.4, 6.35)
- moved C22 1.27 mm to (9.91, 8.64)
- moved C34 1.27 mm to (34.5, 13.2)
- moved R19 1.27 mm to (9.91, 13.2)
- moved R15 0.92 mm to (8.89, 17.0), turned to 180 degrees
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Connections:
- net +3V3: now also IMU.2; no longer IMU.3
- net +5V: now also C41.1, ENCODER.2, HALL1.2, HALL2.2, HALL3.2; no longer ENCODER.1, HALL1.1, HALL2.1, HALL3.1
- net GND: now also C41.2, ENCODER.1, HALL1.1, HALL2.1, HALL3.1, IMU.1; no longer ENCODER.2, HALL1.2, HALL2.2, HALL3.2, IMU.4
- net IMUSCL: now also IMU.3; no longer IMU.1
- net IMUSDA: now also IMU.4; no longer IMU.2
Routing:
- net N$3: track 0.00 -> 14.4 mm
- net N$7: track 0.00 -> 14.2 mm
- net GND: track 100.8 -> 101.6 mm
- net N$2: track 14.5 -> 15.1 mm
- net +5V: track 27.1 -> 26.8 mm, vias 18 -> 19
Other:
- board text added: "PiCar Control Board v2.1 - June 2017 WashU ESE Dept"
- board text removed: "Pi Car Control Board v2.1 WashU ESE Dept May 2017"

Commit message: before autoroute
Parts:
- moved U12 0.92 mm to (3.56, 19.1)
- moved LED1 0.80 mm to (2.03, 19.1), turned to 90 degrees
- moved R48 0.57 mm to (9.40, 10.7)
- moved C22 0.57 mm to (9.40, 8.38)
- moved R19 0.57 mm to (9.40, 13.0)
- turned C31 to 180 degrees
Routing:
- net +3V3: track 0.00 -> 141.8 mm, vias 0 -> 5
- net GND: track 101.6 -> 141.7 mm, vias 33 -> 44
- net +5V: track 26.8 -> 58.2 mm, vias 19 -> 26
- net ATPB0: track 0.00 -> 14.4 mm
- net ATPB2: track 0.00 -> 9.33 mm
- net ATPB1: track 0.00 -> 8.46 mm
- net N$16: track 0.00 -> 4.61 mm
- net ATRESET: track 0.00 -> 4.58 mm
- net N$25: track 0.00 -> 3.84 mm
- net N$26: track 7.22 -> 9.98 mm
- net N$24: track 7.73 -> 10.5 mm
- net N$5: track 7.25 -> 9.98 mm
- net N$22: track 0.00 -> 2.62 mm, vias 0 -> 1
- net VBATT: track 0.00 -> 1.58 mm, vias 0 -> 1
- net ATADC2: track 9.32 -> 9.90 mm
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
Commit message: routed board
Routing:
- net ATRESET: track 4.58 -> 77.2 mm, vias 0 -> 3
- net ATPB1: track 8.46 -> 80.4 mm, vias 0 -> 4
- net ATPB2: track 9.33 -> 78.4 mm, vias 0 -> 5
- net ATICP1: track 0.00 -> 68.8 mm
- net RPILEDG: track 0.00 -> 61.9 mm, vias 0 -> 2
- net ATPB0: track 14.4 -> 74.2 mm, vias 0 -> 3
- net RPILEDB: track 0.00 -> 53.9 mm, vias 0 -> 2
- net ATPF7: track 0.00 -> 52.2 mm, vias 0 -> 2
- net IMUSCL: track 0.00 -> 50.7 mm, vias 0 -> 1
- net ATOC1C: track 0.00 -> 44.3 mm
- net ATMISO: track 0.00 -> 43.6 mm, vias 0 -> 1
- net RPIROMSCL: track 0.00 -> 42.0 mm
- net ATPD5: track 0.00 -> 41.0 mm, vias 0 -> 3
- net ATTX1: track 0.00 -> 40.4 mm, vias 0 -> 2
- net IMUSDA: track 0.00 -> 40.3 mm, vias 0 -> 1
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