File: hw/motorcontrol/v2.1/motorcontrol.sch (EAGLE design)
At the start: 117 parts, among them U1 BTN8982TA, U10 SN74LV4T125, U11 SI2333CDS-T1-GE3, U12 BSS138BKS, U13 BSS138BKS, U2 BTN8982TA, U3 BTN8982TA, U4 CAT24C32, U5 SN74LV4T125, U6 MMDT5401, U7 PTR08060W, U8 IPD90P03P4L-04, U9 ATMEGA32U4

Commit message: fixed error in connection between IS U3 and ATADC4
Connections:
- removed net ATADC2: C9.1, R10.2, U3.IS
- removed net ATPD6: U9.PD6(T1/!OC4D!/ADC9)
- removed net ATPD7: U9.PD7(T0/OC4D/ADC10)
- net ATADC4: now also C9.1, R10.2, U3.IS
Changed lines of the file:
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@@
 <?xml version="1.0" encoding="utf-8"?>
 <!DOCTYPE eagle SYSTEM "eagle.dtd">
-<eagle version="7.7.0">
+<eagle version="8.2.1">
 <drawing>
 <settings>
@@
 <pinref part="R45" gate="G$1" pin="1"/>
 <wire x1="53.34" y1="231.14" x2="53.34" y2="228.6" width="0.1524" layer="91"/>
-<label x="7.62" y="129.54" size="1.778" layer="95"/>
 <wire x1="53.34" y1="228.6" x2="48.26" y2="228.6" width="0.1524" layer="91"/>
 <label x="63.5" y="228.6" size="1.778" layer="95"/>
@@
 </segment>
 <segment>
+<pinref part="J1" gate="A" pin="IDSDA"/>
 <wire x1="25.4" y1="129.54" x2="7.62" y2="129.54" width="0.1524" layer="91"/>
-<pinref part="J1" gate="A" pin="IDSDA"/>
+<label x="7.62" y="129.54" size="1.778" layer="95"/>
 </segment>
 </net>
@@
 <label x="200.66" y="220.98" size="1.778" layer="95"/>
 </segment>
+<segment>
+<pinref part="R10" gate="G$1" pin="2"/>
+<wire x1="177.8" y1="55.88" x2="177.8" y2="58.42" width="0.1524" layer="91"/>
+<label x="180.34" y="58.42" size="1.778" layer="95"/>
+<pinref part="U3" gate="G$1" pin="IS"/>
+<wire x1="208.28" y1="58.42" x2="177.8" y2="58.42" width="0.1524" layer="91"/>
+<pinref part="C9" gate="G$1" pin="1"/>
+<wire x1="172.72" y1="55.88" x2="172.72" y2="58.42" width="0.1524" layer="91"/>
+<wire x1="172.72" y1="58.42" x2="177.8" y2="58.42" width="0.1524" layer="91"/>
+<junction x="177.8" y="58.42"/>
+</segment>
 </net>
 <net name="ATPF5" class="0">
@@
 <junction x="340.36" y="167.64"/>
 <label x="327.66" y="167.64" size="1.778" layer="95"/>
-</segment>
-</net>
-<net name="ATPD7" class="0">
-<segment>
-<pinref part="U9" gate="G$1" pin="PD7(T0/OC4D/ADC10)"/>
-<wire x1="198.12" y1="170.18" x2="203.2" y2="170.18" width="0.1524" layer="91"/>
-<label x="200.66" y="170.18" size="1.778" layer="95"/>
-</segment>
-</net>
-<net name="ATPD6" class="0">
-<segment>
-<pinref part="U9" gate="G$1" pin="PD6(T1/!OC4D!/ADC9)"/>
-<wire x1="198.12" y1="167.64" x2="203.2" y2="167.64" width="0.1524" layer="91"/>
-<label x="200.66" y="167.64" size="1.778" layer="95"/>
 </segment>
 </net>
@@
 </segment>
 </net>
-<net name="ATADC2" class="0">
-<segment>
-<pinref part="R10" gate="G$1" pin="2"/>
-<wire x1="177.8" y1="55.88" x2="177.8" y2="58.42" width="0.1524" layer="91"/>
-<label x="180.34" y="58.42" size="1.778" layer="95"/>
-<pinref part="U3" gate="G$1" pin="IS"/>
-<wire x1="208.28" y1="58.42" x2="177.8" y2="58.42" width="0.1524" layer="91"/>
-<pinref part="C9" gate="G$1" pin="1"/>
-<wire x1="172.72" y1="55.88" x2="172.72" y2="58.42" width="0.1524" layer="91"/>
-<wire x1="172.72" y1="58.42" x2="177.8" y2="58.42" width="0.1524" layer="91"/>
-<junction x="177.8" y="58.42"/>
-</segment>
-</net>
